File: kicad/register.sch (KiCad schematic (older format))
At the start: 2 parts, among them U8 74HCT574, U9 74HC245

Commit message: Fix bug
Connections:
- wire segments 22 -> 24
Changed lines of the file:
@@
 $Descr A4 11693 8268
 encoding utf-8
-Sheet 12 15
+Sheet 10 15
 Title ""
 Date ""
@@
 AR Path="/5AFD5CE2/5AFCB55D/5AFDC209" Ref="#PWR0148"  Part="1"
 AR Path="/5AFD5CE2/5AFCB584/5AFDC209" Ref="#PWR0154"  Part="1"
-F 0 "#PWR0154" H 1500 2450 50  0001 C CNN
+F 0 "#PWR0142" H 1500 2450 50  0001 C CNN
 F 1 "GND" H 1505 2527 50  0000 C CNN
 F 2 "" H 1500 2700 50  0001 C CNN
@@
 AR Path="/5AFD5CE2/5AFCB55D/5AFDC20F" Ref="#PWR0149"  Part="1"
 AR Path="/5AFD5CE2/5AFCB584/5AFDC20F" Ref="#PWR0155"  Part="1"
-F 0 "#PWR0155" H 1500 950 50  0001 C CNN
+F 0 "#PWR0143" H 1500 950 50  0001 C CNN
 F 1 "VCC" H 1517 1273 50  0000 C CNN
 F 2 "" H 1500 1100 50  0001 C CNN
@@
 AR Path="/5AFD5CE2/5AFCB55D/5AFDC225" Ref="#PWR0150"  Part="1"
 AR Path="/5AFD5CE2/5AFCB584/5AFDC225" Ref="#PWR0156"  Part="1"
-F 0 "#PWR0156" H 1000 2150 50  0001 C CNN
+F 0 "#PWR0144" H 1000 2150 50  0001 C CNN
 F 1 "GND" H 1005 2227 50  0000 C CNN
 F 2 "" H 1000 2400 50  0001 C CNN
@@
 AR Path="/5AFD5CE2/5AFCB55D/5AFDC23D" Ref="#PWR0151"  Part="1"
 AR Path="/5AFD5CE2/5AFCB584/5AFDC23D" Ref="#PWR0157"  Part="1"
-F 0 "#PWR0157" H 3300 2450 50  0001 C CNN
+F 0 "#PWR0145" H 3300 2450 50  0001 C CNN
 F 1 "GND" H 3305 2527 50  0000 C CNN
 F 2 "" H 3300 2700 50  0001 C CNN
@@
 AR Path="/5AFD5CE2/5AFCB55D/5AFDC243" Ref="#PWR0152"  Part="1"
 AR Path="/5AFD5CE2/5AFCB584/5AFDC243" Ref="#PWR0158"  Part="1"
-F 0 "#PWR0158" H 2800 2150 50  0001 C CNN
+F 0 "#PWR0146" H 2800 2150 50  0001 C CNN
 F 1 "VCC" H 2817 2473 50  0000 C CNN
 F 2 "" H 2800 2300 50  0001 C CNN
@@
 AR Path="/5AFD5CE2/5AFCB55D/5AFDC249" Ref="#PWR0153"  Part="1"
 AR Path="/5AFD5CE2/5AFCB584/5AFDC249" Ref="#PWR0159"  Part="1"
-F 0 "#PWR0159" H 3300 950 50  0001 C CNN
+F 0 "#PWR0147" H 3300 950 50  0001 C CNN
 F 1 "VCC" H 3317 1273 50  0000 C CNN
 F 2 "" H 3300 1100 50  0001 C CNN
@@
 	2750 2100 2000 2100
 Wire Wire Line
-	2000 1800 2800 1800
+	2000 1800 2450 1800
 Text HLabel 2800 2400 0    50   Input ~ 0
 REG_OUT
@@
 Text HLabel 3800 2100 2    50   Input ~ 0
 O7
+Wire Wire Line
+	2450 1300 2450 1800
+Connection ~ 2450 1800
+Wire Wire Line
+	2450 1800 2800 1800
 $EndSCHEMATC

Commit message: Add micro-usb
Changed lines of the file:
@@
 $Descr A4 11693 8268
 encoding utf-8
-Sheet 10 15
+Sheet 12 15
 Title ""
 Date ""
@@
 AR Path="/5AFD5CE2/5AFDC184/5AFDC202" Ref="U8"  Part="1"
 AR Path="/5AFD5CE2/5AFDFFA6/5AFDC202" Ref="U10"  Part="1"
-AR Path="/5AFD5CE2/5AFCB536/5AFDC202" Ref="U8"  Part="1"
-AR Path="/5AFD5CE2/5AFCB55D/5AFDC202" Ref="U8"  Part="1"
-AR Path="/5AFD5CE2/5AFCB584/5AFDC202" Ref="U8"  Part="1"
-F 0 "U8" H 1600 2600 50  0000 C CNN
+AR Path="/5AFD5CE2/5AFCB536/5AFDC202" Ref="U12"  Part="1"
+AR Path="/5AFD5CE2/5AFCB55D/5AFDC202" Ref="U14"  Part="1"
+AR Path="/5AFD5CE2/5AFCB584/5AFDC202" Ref="U16"  Part="1"
+F 0 "U16" H 1600 2600 50  0000 C CNN
 F 1 "74HCT574" H 1500 1600 50  0000 C CNN
 F 2 "Package_DIP:DIP-20_W7.62mm_Socket" H 1500 1900 50  0001 C CNN
@@
 AR Path="/5AFD5CE2/5AFDC184/5AFDC209" Ref="#PWR0130"  Part="1"
 AR Path="/5AFD5CE2/5AFDFFA6/5AFDC209" Ref="#PWR0136"  Part="1"
-AR Path="/5AFD5CE2/5AFCB536/5AFDC209" Ref="#PWR0142"  Part="1"
-AR Path="/5AFD5CE2/5AFCB55D/5AFDC209" Ref="#PWR0148"  Part="1"
-AR Path="/5AFD5CE2/5AFCB584/5AFDC209" Ref="#PWR0154"  Part="1"
-F 0 "#PWR0142" H 1500 2450 50  0001 C CNN
+AR Path="/5AFD5CE2/5AFCB536/5AFDC209" Ref="#PWR020"  Part="1"
+AR Path="/5AFD5CE2/5AFCB55D/5AFDC209" Ref="#PWR028"  Part="1"
+AR Path="/5AFD5CE2/5AFCB584/5AFDC209" Ref="#PWR034"  Part="1"
+F 0 "#PWR034" H 1500 2450 50  0001 C CNN
 F 1 "GND" H 1505 2527 50  0000 C CNN
 F 2 "" H 1500 2700 50  0001 C CNN
@@
 AR Path="/5AFD5CE2/5AFDC184/5AFDC20F" Ref="#PWR0131"  Part="1"
 AR Path="/5AFD5CE2/5AFDFFA6/5AFDC20F" Ref="#PWR0137"  Part="1"
-AR Path="/5AFD5CE2/5AFCB536/5AFDC20F" Ref="#PWR0143"  Part="1"
-AR Path="/5AFD5CE2/5AFCB55D/5AFDC20F" Ref="#PWR0149"  Part="1"
-AR Path="/5AFD5CE2/5AFCB584/5AFDC20F" Ref="#PWR0155"  Part="1"
-F 0 "#PWR0143" H 1500 950 50  0001 C CNN
+AR Path="/5AFD5CE2/5AFCB536/5AFDC20F" Ref="#PWR018"  Part="1"
+AR Path="/5AFD5CE2/5AFCB55D/5AFDC20F" Ref="#PWR027"  Part="1"
+AR Path="/5AFD5CE2/5AFCB584/5AFDC20F" Ref="#PWR033"  Part="1"
+F 0 "#PWR033" H 1500 950 50  0001 C CNN
 F 1 "VCC" H 1517 1273 50  0000 C CNN
 F 2 "" H 1500 1100 50  0001 C CNN
@@
 AR Path="/5AFD5CE2/5AFDC184/5AFDC21E" Ref="U9"  Part="1"
 AR Path="/5AFD5CE2/5AFDFFA6/5AFDC21E" Ref="U11"  Part="1"
-AR Path="/5AFD5CE2/5AFCB536/5AFDC21E" Ref="U9"  Part="1"
-AR Path="/5AFD5CE2/5AFCB55D/5AFDC21E" Ref="U9"  Part="1"
-AR Path="/5AFD5CE2/5AFCB584/5AFDC21E" Ref="U9"  Part="1"
-F 0 "U9" H 3400 2600 50  0000 C CNN
+AR Path="/5AFD5CE2/5AFCB536/5AFDC21E" Ref="U13"  Part="1"
+AR Path="/5AFD5CE2/5AFCB55D/5AFDC21E" Ref="U15"  Part="1"
+AR Path="/5AFD5CE2/5AFCB584/5AFDC21E" Ref="U17"  Part="1"
+F 0 "U17" H 3400 2600 50  0000 C CNN
 F 1 "74HC245" H 3350 1600 50  0000 C CNN
 F 2 "Package_DIP:DIP-20_W7.62mm_Socket" H 3300 1900 50  0001 C CNN
@@
 AR Path="/5AFD5CE2/5AFDC184/5AFDC225" Ref="#PWR0132"  Part="1"
 AR Path="/5AFD5CE2/5AFDFFA6/5AFDC225" Ref="#PWR0138"  Part="1"
-AR Path="/5AFD5CE2/5AFCB536/5AFDC225" Ref="#PWR0144"  Part="1"
-AR Path="/5AFD5CE2/5AFCB55D/5AFDC225" Ref="#PWR0150"  Part="1"
-AR Path="/5AFD5CE2/5AFCB584/5AFDC225" Ref="#PWR0156"  Part="1"
-F 0 "#PWR0144" H 1000 2150 50  0001 C CNN
+AR Path="/5AFD5CE2/5AFCB536/5AFDC225" Ref="#PWR016"  Part="1"
+AR Path="/5AFD5CE2/5AFCB55D/5AFDC225" Ref="#PWR026"  Part="1"
+AR Path="/5AFD5CE2/5AFCB584/5AFDC225" Ref="#PWR032"  Part="1"
+F 0 "#PWR032" H 1000 2150 50  0001 C CNN
 F 1 "GND" H 1005 2227 50  0000 C CNN
 F 2 "" H 1000 2400 50  0001 C CNN
@@
 AR Path="/5AFD5CE2/5AFDC184/5AFDC23D" Ref="#PWR0133"  Part="1"
 AR Path="/5AFD5CE2/5AFDFFA6/5AFDC23D" Ref="#PWR0139"  Part="1"
-AR Path="/5AFD5CE2/5AFCB536/5AFDC23D" Ref="#PWR0145"  Part="1"
-AR Path="/5AFD5CE2/5AFCB55D/5AFDC23D" Ref="#PWR0151"  Part="1"
-AR Path="/5AFD5CE2/5AFCB584/5AFDC23D" Ref="#PWR0157"  Part="1"
-F 0 "#PWR0145" H 3300 2450 50  0001 C CNN
+AR Path="/5AFD5CE2/5AFCB536/5AFDC23D" Ref="#PWR025"  Part="1"
+AR Path="/5AFD5CE2/5AFCB55D/5AFDC23D" Ref="#PWR031"  Part="1"
+AR Path="/5AFD5CE2/5AFCB584/5AFDC23D" Ref="#PWR037"  Part="1"
+F 0 "#PWR037" H 3300 2450 50  0001 C CNN
 F 1 "GND" H 3305 2527 50  0000 C CNN
 F 2 "" H 3300 2700 50  0001 C CNN
@@
 AR Path="/5AFD5CE2/5AFDC184/5AFDC243" Ref="#PWR0134"  Part="1"
 AR Path="/5AFD5CE2/5AFDFFA6/5AFDC243" Ref="#PWR0140"  Part="1"
-AR Path="/5AFD5CE2/5AFCB536/5AFDC243" Ref="#PWR0146"  Part="1"
-AR Path="/5AFD5CE2/5AFCB55D/5AFDC243" Ref="#PWR0152"  Part="1"
-AR Path="/5AFD5CE2/5AFCB584/5AFDC243" Ref="#PWR0158"  Part="1"
-F 0 "#PWR0146" H 2800 2150 50  0001 C CNN
+AR Path="/5AFD5CE2/5AFCB536/5AFDC243" Ref="#PWR023"  Part="1"
+AR Path="/5AFD5CE2/5AFCB55D/5AFDC243" Ref="#PWR029"  Part="1"
+AR Path="/5AFD5CE2/5AFCB584/5AFDC243" Ref="#PWR035"  Part="1"
+F 0 "#PWR035" H 2800 2150 50  0001 C CNN
 F 1 "VCC" H 2817 2473 50  0000 C CNN
 F 2 "" H 2800 2300 50  0001 C CNN
@@
 AR Path="/5AFD5CE2/5AFDC184/5AFDC249" Ref="#PWR0135"  Part="1"
 AR Path="/5AFD5CE2/5AFDFFA6/5AFDC249" Ref="#PWR0141"  Part="1"
-AR Path="/5AFD5CE2/5AFCB536/5AFDC249" Ref="#PWR0147"  Part="1"
-AR Path="/5AFD5CE2/5AFCB55D/5AFDC249" Ref="#PWR0153"  Part="1"
-AR Path="/5AFD5CE2/5AFCB584/5AFDC249" Ref="#PWR0159"  Part="1"
-F 0 "#PWR0147" H 3300 950 50  0001 C CNN
+AR Path="/5AFD5CE2/5AFCB536/5AFDC249" Ref="#PWR024"  Part="1"
+AR Path="/5AFD5CE2/5AFCB55D/5AFDC249" Ref="#PWR030"  Part="1"
+AR Path="/5AFD5CE2/5AFCB584/5AFDC249" Ref="#PWR036"  Part="1"
+F 0 "#PWR036" H 3300 950 50  0001 C CNN
 F 1 "VCC" H 3317 1273 50  0000 C CNN
 F 2 "" H 3300 1100 50  0001 C CNN

Commit message: Remove register LEDs
Connections:
- wire segments 24 -> 8
Other:
- moved on the sheet: U19
Changed lines of the file:
@@
 $Descr A4 11693 8268
 encoding utf-8
-Sheet 12 15
+Sheet 11 11
 Title ""
 Date ""
@@
 AR Path="/5AFD5CE2/5AFCB55D/5AFDC202" Ref="U14"  Part="1"
 AR Path="/5AFD5CE2/5AFCB584/5AFDC202" Ref="U16"  Part="1"
-F 0 "U16" H 1600 2600 50  0000 C CNN
+AR Path="/5AFD5CE2/5AFD86BE/5AFDC202" Ref="U18"  Part="1"
+F 0 "U18" H 1600 2600 50  0000 C CNN
 F 1 "74HCT574" H 1500 1600 50  0000 C CNN
 F 2 "Package_DIP:DIP-20_W7.62mm_Socket" H 1500 1900 50  0001 C CNN
@@
 AR Path="/5AFD5CE2/5AFCB55D/5AFDC209" Ref="#PWR028"  Part="1"
 AR Path="/5AFD5CE2/5AFCB584/5AFDC209" Ref="#PWR034"  Part="1"
-F 0 "#PWR034" H 1500 2450 50  0001 C CNN
+AR Path="/5AFD5CE2/5AFD86BE/5AFDC209" Ref="#PWR0142"  Part="1"
+F 0 "#PWR0142" H 1500 2450 50  0001 C CNN
 F 1 "GND" H 1505 2527 50  0000 C CNN
 F 2 "" H 1500 2700 50  0001 C CNN
@@
 AR Path="/5AFD5CE2/5AFCB55D/5AFDC20F" Ref="#PWR027"  Part="1"
 AR Path="/5AFD5CE2/5AFCB584/5AFDC20F" Ref="#PWR033"  Part="1"
-F 0 "#PWR033" H 1500 950 50  0001 C CNN
+AR Path="/5AFD5CE2/5AFD86BE/5AFDC20F" Ref="#PWR0143"  Part="1"
+F 0 "#PWR0143" H 1500 950 50  0001 C CNN
 F 1 "VCC" H 1517 1273 50  0000 C CNN
 F 2 "" H 1500 1100 50  0001 C CNN
@@
 L 74xx:74HC245 U?
 U 1 1 5AFDC21E
-P 3300 1900
+P 2750 1900
 AR Path="/5AFD5CE2/5AFDC21E" Ref="U?"  Part="1"
 AR Path="/5AFD5CE2/5AFDC184/5AFDC21E" Ref="U9"  Part="1"
@@
 AR Path="/5AFD5CE2/5AFCB55D/5AFDC21E" Ref="U15"  Part="1"
 AR Path="/5AFD5CE2/5AFCB584/5AFDC21E" Ref="U17"  Part="1"
-F 0 "U17" H 3400 2600 50  0000 C CNN
-F 1 "74HC245" H 3350 1600 50  0000 C CNN
-F 2 "Package_DIP:DIP-20_W7.62mm_Socket" H 3300 1900 50  0001 C CNN
-F 3 "http://www.ti.com/lit/gpn/sn74HC245" H 3300 1900 50  0001 C CNN
-	1    3300 1900
+AR Path="/5AFD5CE2/5AFD86BE/5AFDC21E" Ref="U19"  Part="1"
+F 0 "U19" H 2850 2600 50  0000 C CNN
+F 1 "74HC245" H 2800 1600 50  0000 C CNN
+F 2 "Package_DIP:DIP-20_W7.62mm_Socket" H 2750 1900 50  0001 C CNN
+F 3 "http://www.ti.com/lit/gpn/sn74HC245" H 2750 1900 50  0001 C CNN
+	1    2750 1900
 	1    0    0    -1
 $EndComp
@@
 AR Path="/5AFD5CE2/5AFCB55D/5AFDC225" Ref="#PWR026"  Part="1"
 AR Path="/5AFD5CE2/5AFCB584/5AFDC225" Ref="#PWR032"  Part="1"
-F 0 "#PWR032" H 1000 2150 50  0001 C CNN
+AR Path="/5AFD5CE2/5AFD86BE/5AFDC225" Ref="#PWR0144"  Part="1"
+F 0 "#PWR0144" H 1000 2150 50  0001 C CNN
 F 1 "GND" H 1005 2227 50  0000 C CNN
 F 2 "" H 1000 2400 50  0001 C CNN
@@
 	1    0    0    -1
 $EndComp
-$Sheet
-S 1950 750  900  550
-U 5AFDC22F
-F0 "Reg Leds" 50
-F1 "bus_leds.sch" 50
-F2 "I0" I B 2050 1300 50
-F3 "I1" I B 2150 1300 50
-F4 "I2" I B 2250 1300 50
-F5 "I3" I B 2350 1300 50
-F6 "I4" I B 2450 1300 50
-F7 "I5" I B 2550 1300 50
-F8 "I6" I B 2650 1300 50
-F9 "I7" I B 2750 1300 50
-$EndSheet
-Wire Wire Line
-	2000 1400 2050 1400
-Wire Wire Line
-	2000 1500 2150 1500
-Wire Wire Line
-	2000 1600 2250 1600
-Wire Wire Line
-	2000 1700 2350 1700
-Wire Wire Line
-	2800 1900 2550 1900
-Wire Wire Line
-	2000 2000 2650 2000
-Wire Wire Line
-	2800 2100 2750 2100
 $Comp
 L power:GND #PWR0133
 U 1 1 5AFDC23D
-P 3300 2700
+P 2750 2700
 AR Path="/5AFD5CE2/5AFDC184/5AFDC23D" Ref="#PWR0133"  Part="1"
 AR Path="/5AFD5CE2/5AFDFFA6/5AFDC23D" Ref="#PWR0139"  Part="1"
@@
 AR Path="/5AFD5CE2/5AFCB55D/5AFDC23D" Ref="#PWR031"  Part="1"
 AR Path="/5AFD5CE2/5AFCB584/5AFDC23D" Ref="#PWR037"  Part="1"
-F 0 "#PWR037" H 3300 2450 50  0001 C CNN
-F 1 "GND" H 3305 2527 50  0000 C CNN
-F 2 "" H 3300 2700 50  0001 C CNN
-F 3 "" H 3300 2700 50  0001 C CNN
-	1    3300 2700
+AR Path="/5AFD5CE2/5AFD86BE/5AFDC23D" Ref="#PWR0145"  Part="1"
+F 0 "#PWR0145" H 2750 2450 50  0001 C CNN
+F 1 "GND" H 2755 2527 50  0000 C CNN
+F 2 "" H 2750 2700 50  0001 C CNN
+F 3 "" H 2750 2700 50  0001 C CNN
+	1    2750 2700
 	1    0    0    -1
 $EndComp
@@
 L power:VCC #PWR0134
 U 1 1 5AFDC243
-P 2800 2300
+P 2250 2300
 AR Path="/5AFD5CE2/5AFDC184/5AFDC243" Ref="#PWR0134"  Part="1"
 AR Path="/5AFD5CE2/5AFDFFA6/5AFDC243" Ref="#PWR0140"  Part="1"
@@
 AR Path="/5AFD5CE2/5AFCB55D/5AFDC243" Ref="#PWR029"  Part="1"
 AR Path="/5AFD5CE2/5AFCB584/5AFDC243" Ref="#PWR035"  Part="1"
-F 0 "#PWR035" H 2800 2150 50  0001 C CNN
-F 1 "VCC" H 2817 2473 50  0000 C CNN
-F 2 "" H 2800 2300 50  0001 C CNN
-F 3 "" H 2800 2300 50  0001 C CNN
-	1    2800 2300
+AR Path="/5AFD5CE2/5AFD86BE/5AFDC243" Ref="#PWR0146"  Part="1"
+F 0 "#PWR0146" H 2250 2150 50  0001 C CNN
+F 1 "VCC" H 2267 2473 50  0000 C CNN
+F 2 "" H 2250 2300 50  0001 C CNN
+F 3 "" H 2250 2300 50  0001 C CNN
+	1    2250 2300
 	0    -1   -1   0
 $EndComp
@@
 L power:VCC #PWR0135
 U 1 1 5AFDC249
-P 3300 1100
+P 2750 1100
 AR Path="/5AFD5CE2/5AFDC184/5AFDC249" Ref="#PWR0135"  Part="1"
 AR Path="/5AFD5CE2/5AFDFFA6/5AFDC249" Ref="#PWR0141"  Part="1"
@@
 AR Path="/5AFD5CE2/5AFCB55D/5AFDC249" Ref="#PWR030"  Part="1"
 AR Path="/5AFD5CE2/5AFCB584/5AFDC249" Ref="#PWR036"  Part="1"
-F 0 "#PWR036" H 3300 950 50  0001 C CNN
-F 1 "VCC" H 3317 1273 50  0000 C CNN
-F 2 "" H 3300 1100 50  0001 C CNN
-F 3 "" H 3300 1100 50  0001 C CNN
-	1    3300 1100
-	1    0    0    -1
-$EndComp
-Wire Wire Line
-	2050 1300 2050 1400
-Connection ~ 2050 1400
-Wire Wire Line
-	2050 1400 2800 1400
-Wire Wire Line
-	2150 1300 2150 1500
-Connection ~ 2150 1500
-Wire Wire Line
-	2150 1500 2800 1500
-Wire Wire Line
-	2250 1600 2250 1300
-Connection ~ 2250 1600
-Wire Wire Line
-	2250 1600 2800 1600
-Wire Wire Line
-	2350 1300 2350 1700
-Connection ~ 2350 1700
-Wire Wire Line
-	2350 1700 2800 1700
-Wire Wire Line
-	2550 1300 2550 1900
-Connection ~ 2550 1900
-Wire Wire Line
-	2550 1900 2000 1900
-Wire Wire Line
-	2650 2000 2650 1300
-Connection ~ 2650 2000
-Wire Wire Line
-	2650 2000 2800 2000
-Wire Wire Line
-	2750 1300 2750 2100
-Connection ~ 2750 2100
-Wire Wire Line
-	2750 2100 2000 2100
-Wire Wire Line
-	2000 1800 2450 1800
-Text HLabel 2800 2400 0    50   Input ~ 0
+AR Path="/5AFD5CE2/5AFD86BE/5AFDC249" Ref="#PWR0147"  Part="1"
+F 0 "#PWR0147" H 2750 950 50  0001 C CNN
+F 1 "VCC" H 2767 1273 50  0000 C CNN
+F 2 "" H 2750 1100 50  0001 C CNN
+F 3 "" H 2750 1100 50  0001 C CNN
+	1    2750 1100
+	1    0    0    -1
+$EndComp
+Text HLabel 2250 2400 0    50   Input ~ 0
 REG_OUT
-Text HLabel 3800 1400 2    50   Input ~ 0
+Text HLabel 3250 1400 2    50   Input ~ 0
 O0
-Text HLabel 3800 1500 2    50   Input ~ 0
+Text HLabel 3250 1500 2    50   Input ~ 0
 O1
-Text HLabel 3800 1600 2    50   Input ~ 0
+Text HLabel 3250 1600 2    50   Input ~ 0
 O2
-Text HLabel 3800 1700 2    50   Input ~ 0
+Text HLabel 3250 1700 2    50   Input ~ 0
 O3
-Text HLabel 3800 1800 2    50   Input ~ 0
+Text HLabel 3250 1800 2    50   Input ~ 0
 O4
-Text HLabel 3800 1900 2    50   Input ~ 0
+Text HLabel 3250 1900 2    50   Input ~ 0
 O5
-Text HLabel 3800 2000 2    50   Input ~ 0
+Text HLabel 3250 2000 2    50   Input ~ 0
 O6
-Text HLabel 3800 2100 2    50   Input ~ 0
+Text HLabel 3250 2100 2    50   Input ~ 0
 O7
 Wire Wire Line
-	2450 1300 2450 1800
-Connection ~ 2450 1800
-Wire Wire Line
-	2450 1800 2800 1800
+	2000 1400 2250 1400
+Wire Wire Line
+	2000 1500 2250 1500
+Wire Wire Line
+	2000 1600 2250 1600
+Wire Wire Line
+	2000 1700 2250 1700
+Wire Wire Line
+	2000 1800 2250 1800
+Wire Wire Line
+	2000 1900 2250 1900
+Wire Wire Line
+	2000 2000 2250 2000
+Wire Wire Line
+	2000 2100 2250 2100
 $EndSCHEMATC

Commit message: Remove bus transceivers from registers, as they are no longer connected to LEDs.
Parts:
- removed U9: 74HC245, Package_DIP:DIP-20_W7.62mm_Socket, symbol 74xx:74HC245
Connections:
- wire segments 8 -> 0
Changed lines of the file:
@@
 $Descr A4 11693 8268
 encoding utf-8
-Sheet 11 11
+Sheet 6 11
 Title ""
 Date ""
@@
 AR Path="/5AFD5CE2/5AFCB584/5AFDC202" Ref="U16"  Part="1"
 AR Path="/5AFD5CE2/5AFD86BE/5AFDC202" Ref="U18"  Part="1"
-F 0 "U18" H 1600 2600 50  0000 C CNN
+F 0 "U8" H 1600 2600 50  0000 C CNN
 F 1 "74HCT574" H 1500 1600 50  0000 C CNN
 F 2 "Package_DIP:DIP-20_W7.62mm_Socket" H 1500 1900 50  0001 C CNN
@@
 Text HLabel 1000 2100 0    50   Input ~ 0
 I7
-$Comp
-L 74xx:74HC245 U?
-U 1 1 5AFDC21E
-P 2750 1900
-AR Path="/5AFD5CE2/5AFDC21E" Ref="U?"  Part="1"
-AR Path="/5AFD5CE2/5AFDC184/5AFDC21E" Ref="U9"  Part="1"
-AR Path="/5AFD5CE2/5AFDFFA6/5AFDC21E" Ref="U11"  Part="1"
-AR Path="/5AFD5CE2/5AFCB536/5AFDC21E" Ref="U13"  Part="1"
-AR Path="/5AFD5CE2/5AFCB55D/5AFDC21E" Ref="U15"  Part="1"
-AR Path="/5AFD5CE2/5AFCB584/5AFDC21E" Ref="U17"  Part="1"
-AR Path="/5AFD5CE2/5AFD86BE/5AFDC21E" Ref="U19"  Part="1"
-F 0 "U19" H 2850 2600 50  0000 C CNN
-F 1 "74HC245" H 2800 1600 50  0000 C CNN
-F 2 "Package_DIP:DIP-20_W7.62mm_Socket" H 2750 1900 50  0001 C CNN
-F 3 "http://www.ti.com/lit/gpn/sn74HC245" H 2750 1900 50  0001 C CNN
-	1    2750 1900
-	1    0    0    -1
-$EndComp
-$Comp
-L power:GND #PWR0132
-U 1 1 5AFDC225
-P 1000 2400
-AR Path="/5AFD5CE2/5AFDC184/5AFDC225" Ref="#PWR0132"  Part="1"
-AR Path="/5AFD5CE2/5AFDFFA6/5AFDC225" Ref="#PWR0138"  Part="1"
-AR Path="/5AFD5CE2/5AFCB536/5AFDC225" Ref="#PWR016"  Part="1"
-AR Path="/5AFD5CE2/5AFCB55D/5AFDC225" Ref="#PWR026"  Part="1"
-AR Path="/5AFD5CE2/5AFCB584/5AFDC225" Ref="#PWR032"  Part="1"
-AR Path="/5AFD5CE2/5AFD86BE/5AFDC225" Ref="#PWR0144"  Part="1"
-F 0 "#PWR0144" H 1000 2150 50  0001 C CNN
-F 1 "GND" H 1005 2227 50  0000 C CNN
-F 2 "" H 1000 2400 50  0001 C CNN
-F 3 "" H 1000 2400 50  0001 C CNN
-	1    1000 2400
-	1    0    0    -1
-$EndComp
-$Comp
-L power:GND #PWR0133
-U 1 1 5AFDC23D
-P 2750 2700
-AR Path="/5AFD5CE2/5AFDC184/5AFDC23D" Ref="#PWR0133"  Part="1"
-AR Path="/5AFD5CE2/5AFDFFA6/5AFDC23D" Ref="#PWR0139"  Part="1"
-AR Path="/5AFD5CE2/5AFCB536/5AFDC23D" Ref="#PWR025"  Part="1"
-AR Path="/5AFD5CE2/5AFCB55D/5AFDC23D" Ref="#PWR031"  Part="1"
-AR Path="/5AFD5CE2/5AFCB584/5AFDC23D" Ref="#PWR037"  Part="1"
-AR Path="/5AFD5CE2/5AFD86BE/5AFDC23D" Ref="#PWR0145"  Part="1"
-F 0 "#PWR0145" H 2750 2450 50  0001 C CNN
-F 1 "GND" H 2755 2527 50  0000 C CNN
-F 2 "" H 2750 2700 50  0001 C CNN
-F 3 "" H 2750 2700 50  0001 C CNN
-	1    2750 2700
-	1    0    0    -1
-$EndComp
-$Comp
-L power:VCC #PWR0134
-U 1 1 5AFDC243
-P 2250 2300
-AR Path="/5AFD5CE2/5AFDC184/5AFDC243" Ref="#PWR0134"  Part="1"
-AR Path="/5AFD5CE2/5AFDFFA6/5AFDC243" Ref="#PWR0140"  Part="1"
-AR Path="/5AFD5CE2/5AFCB536/5AFDC243" Ref="#PWR023"  Part="1"
-AR Path="/5AFD5CE2/5AFCB55D/5AFDC243" Ref="#PWR029"  Part="1"
-AR Path="/5AFD5CE2/5AFCB584/5AFDC243" Ref="#PWR035"  Part="1"
-AR Path="/5AFD5CE2/5AFD86BE/5AFDC243" Ref="#PWR0146"  Part="1"
-F 0 "#PWR0146" H 2250 2150 50  0001 C CNN
-F 1 "VCC" H 2267 2473 50  0000 C CNN
-F 2 "" H 2250 2300 50  0001 C CNN
-F 3 "" H 2250 2300 50  0001 C CNN
-	1    2250 2300
-	0    -1   -1   0
-$EndComp
-$Comp
-L power:VCC #PWR0135
-U 1 1 5AFDC249
-P 2750 1100
-AR Path="/5AFD5CE2/5AFDC184/5AFDC249" Ref="#PWR0135"  Part="1"
-AR Path="/5AFD5CE2/5AFDFFA6/5AFDC249" Ref="#PWR0141"  Part="1"
-AR Path="/5AFD5CE2/5AFCB536/5AFDC249" Ref="#PWR024"  Part="1"
-AR Path="/5AFD5CE2/5AFCB55D/5AFDC249" Ref="#PWR030"  Part="1"
-AR Path="/5AFD5CE2/5AFCB584/5AFDC249" Ref="#PWR036"  Part="1"
-AR Path="/5AFD5CE2/5AFD86BE/5AFDC249" Ref="#PWR0147"  Part="1"
-F 0 "#PWR0147" H 2750 950 50  0001 C CNN
-F 1 "VCC" H 2767 1273 50  0000 C CNN
-F 2 "" H 2750 1100 50  0001 C CNN
-F 3 "" H 2750 1100 50  0001 C CNN
-	1    2750 1100
-	1    0    0    -1
-$EndComp
-Text HLabel 2250 2400 0    50   Input ~ 0
+Text HLabel 1000 2400 0    50   Input ~ 0
 REG_OUT
-Text HLabel 3250 1400 2    50   Input ~ 0
+Text HLabel 2000 1400 2    50   Input ~ 0
 O0
-Text HLabel 3250 1500 2    50   Input ~ 0
+Text HLabel 2000 1500 2    50   Input ~ 0
 O1
-Text HLabel 3250 1600 2    50   Input ~ 0
+Text HLabel 2000 1600 2    50   Input ~ 0
 O2
-Text HLabel 3250 1700 2    50   Input ~ 0
+Text HLabel 2000 1700 2    50   Input ~ 0
 O3
-Text HLabel 3250 1800 2    50   Input ~ 0
+Text HLabel 2000 1800 2    50   Input ~ 0
 O4
-Text HLabel 3250 1900 2    50   Input ~ 0
+Text HLabel 2000 1900 2    50   Input ~ 0
 O5
-Text HLabel 3250 2000 2    50   Input ~ 0
+Text HLabel 2000 2000 2    50   Input ~ 0
 O6
-Text HLabel 3250 2100 2    50   Input ~ 0
+Text HLabel 2000 2100 2    50   Input ~ 0
 O7
-Wire Wire Line
-	2000 1400 2250 1400
-Wire Wire Line
-	2000 1500 2250 1500
-Wire Wire Line
-	2000 1600 2250 1600
-Wire Wire Line
-	2000 1700 2250 1700
-Wire Wire Line
-	2000 1800 2250 1800
-Wire Wire Line
-	2000 1900 2250 1900
-Wire Wire Line
-	2000 2000 2250 2000
-Wire Wire Line
-	2000 2100 2250 2100
 $EndSCHEMATC

Commit message: Add bus transceivers back just for registers A and B, so they can be connected to the ALU. Add ALU to schematic.
Parts:
- added C16: C_Small, Capacitor_THT:C_Disc_D3.0mm_W2.0mm_P2.50mm, symbol Device:C_Small
Connections:
- wire segments 0 -> 4
Changed lines of the file:
@@
 $Descr A4 11693 8268
 encoding utf-8
-Sheet 6 11
+Sheet 6 12
 Title ""
 Date ""
@@
 AR Path="/5AFD5CE2/5AFCB584/5AFDC202" Ref="U16"  Part="1"
 AR Path="/5AFD5CE2/5AFD86BE/5AFDC202" Ref="U18"  Part="1"
-F 0 "U8" H 1600 2600 50  0000 C CNN
+F 0 "U18" H 1600 2600 50  0000 C CNN
 F 1 "74HCT574" H 1500 1600 50  0000 C CNN
 F 2 "Package_DIP:DIP-20_W7.62mm_Socket" H 1500 1900 50  0001 C CNN
@@
 Text HLabel 2000 2100 2    50   Input ~ 0
 O7
+$Comp
+L Device:C_Small C?
+U 1 1 5AFDADFB
+P 2500 1800
+AR Path="/5AFD5CE2/5AFDC184/5AFDADFB" Ref="C?"  Part="1"
+AR Path="/5AFD5CE2/5AFCB536/5AFDADFB" Ref="C16"  Part="1"
+AR Path="/5AFD5CE2/5AFCB55D/5AFDADFB" Ref="C17"  Part="1"
+AR Path="/5AFD5CE2/5AFCB584/5AFDADFB" Ref="C18"  Part="1"
+AR Path="/5AFD5CE2/5AFD86BE/5AFDADFB" Ref="C19"  Part="1"
+F 0 "C19" H 2592 1846 50  0000 L CNN
+F 1 "C_Small" H 2592 1755 50  0000 L CNN
+F 2 "Capacitor_THT:C_Disc_D3.0mm_W2.0mm_P2.50mm" H 2500 1800 50  0001 C CNN
+F 3 "~" H 2500 1800 50  0001 C CNN
+	1    2500 1800
+	1    0    0    -1
+$EndComp
+Wire Wire Line
+	1500 1100 2500 1100
+Wire Wire Line
+	2500 1100 2500 1700
+Connection ~ 1500 1100
+Wire Wire Line
+	2500 1900 2500 2700
+Wire Wire Line
+	2500 2700 1500 2700
+Connection ~ 1500 2700
 $EndSCHEMATC

Commit message: Add display module. Still need to check if it needs resistors.
Changed lines of the file:
@@
 $Descr A4 11693 8268
 encoding utf-8
-Sheet 6 12
+Sheet 14 14
 Title ""
 Date ""
@@
 AR Path="/5AFD5CE2/5AFCB584/5AFDC202" Ref="U16"  Part="1"
 AR Path="/5AFD5CE2/5AFD86BE/5AFDC202" Ref="U18"  Part="1"
-F 0 "U18" H 1600 2600 50  0000 C CNN
+AR Path="/5AFEE19A/5B043D5C/5AFDC202" Ref="U29"  Part="1"
+F 0 "U29" H 1600 2600 50  0000 C CNN
 F 1 "74HCT574" H 1500 1600 50  0000 C CNN
 F 2 "Package_DIP:DIP-20_W7.62mm_Socket" H 1500 1900 50  0001 C CNN
@@
 AR Path="/5AFD5CE2/5AFCB584/5AFDC209" Ref="#PWR034"  Part="1"
 AR Path="/5AFD5CE2/5AFD86BE/5AFDC209" Ref="#PWR0142"  Part="1"
-F 0 "#PWR0142" H 1500 2450 50  0001 C CNN
+AR Path="/5AFEE19A/5B043D5C/5AFDC209" Ref="#PWR0164"  Part="1"
+F 0 "#PWR0164" H 1500 2450 50  0001 C CNN
 F 1 "GND" H 1505 2527 50  0000 C CNN
 F 2 "" H 1500 2700 50  0001 C CNN
@@
 AR Path="/5AFD5CE2/5AFCB584/5AFDC20F" Ref="#PWR033"  Part="1"
 AR Path="/5AFD5CE2/5AFD86BE/5AFDC20F" Ref="#PWR0143"  Part="1"
-F 0 "#PWR0143" H 1500 950 50  0001 C CNN
+AR Path="/5AFEE19A/5B043D5C/5AFDC20F" Ref="#PWR0165"  Part="1"
+F 0 "#PWR0165" H 1500 950 50  0001 C CNN
 F 1 "VCC" H 1517 1273 50  0000 C CNN
 F 2 "" H 1500 1100 50  0001 C CNN
@@
 AR Path="/5AFD5CE2/5AFCB584/5AFDADFB" Ref="C18"  Part="1"
 AR Path="/5AFD5CE2/5AFD86BE/5AFDADFB" Ref="C19"  Part="1"
-F 0 "C19" H 2592 1846 50  0000 L CNN
+AR Path="/5AFEE19A/5B043D5C/5AFDADFB" Ref="C36"  Part="1"
+F 0 "C36" H 2592 1846 50  0000 L CNN
 F 1 "C_Small" H 2592 1755 50  0000 L CNN
 F 2 "Capacitor_THT:C_Disc_D3.0mm_W2.0mm_P2.50mm" H 2500 1800 50  0001 C CNN
