File: kicad/register.sch (KiCad schematic (older format))
At the start: 2 parts, among them U8 74HCT574

Commit message: Update notes. Layout extra clock stuff.
Changed lines of the file:
@@
 AR Path="/5AFD5CE2/5AFD86BE/5AFDC202" Ref="U18"  Part="1"
 AR Path="/5AFEE19A/5B043D5C/5AFDC202" Ref="U29"  Part="1"
-F 0 "U29" H 1600 2600 50  0000 C CNN
+F 0 "U12" H 1600 2600 50  0000 C CNN
 F 1 "74HCT574" H 1500 1600 50  0000 C CNN
 F 2 "Package_DIP:DIP-20_W7.62mm_Socket" H 1500 1900 50  0001 C CNN
@@
 AR Path="/5AFD5CE2/5AFD86BE/5AFDC209" Ref="#PWR0142"  Part="1"
 AR Path="/5AFEE19A/5B043D5C/5AFDC209" Ref="#PWR0164"  Part="1"
-F 0 "#PWR0164" H 1500 2450 50  0001 C CNN
+F 0 "#PWR020" H 1500 2450 50  0001 C CNN
 F 1 "GND" H 1505 2527 50  0000 C CNN
 F 2 "" H 1500 2700 50  0001 C CNN
@@
 AR Path="/5AFD5CE2/5AFD86BE/5AFDC20F" Ref="#PWR0143"  Part="1"
 AR Path="/5AFEE19A/5B043D5C/5AFDC20F" Ref="#PWR0165"  Part="1"
-F 0 "#PWR0165" H 1500 950 50  0001 C CNN
+F 0 "#PWR018" H 1500 950 50  0001 C CNN
 F 1 "VCC" H 1517 1273 50  0000 C CNN
 F 2 "" H 1500 1100 50  0001 C CNN
@@
 AR Path="/5AFD5CE2/5AFD86BE/5AFDADFB" Ref="C19"  Part="1"
 AR Path="/5AFEE19A/5B043D5C/5AFDADFB" Ref="C36"  Part="1"
-F 0 "C36" H 2592 1846 50  0000 L CNN
+F 0 "C16" H 2592 1846 50  0000 L CNN
 F 1 "C_Small" H 2592 1755 50  0000 L CNN
 F 2 "Capacitor_THT:C_Disc_D3.0mm_W2.0mm_P2.50mm" H 2500 1800 50  0001 C CNN
