File: kicad/manual_bus.sch (KiCad schematic (older format))
At the start: 10 parts

Commit message: Think about design. Add A and B registers to schematic and pcb.
Parts:
- R15, R16, R17, R18, R19, R20, R21, R22: renamed from R?; footprint (none) -> Resistor_THT:R_Axial_DIN0207_L6.3mm_D2.5mm_P7.62mm_Horizontal
- SW4: renamed from SW?; footprint (none) -> Button_Switch_THT:SW_DIP_SPSTx08_Slide_9.78x22.5mm_W7.62mm_P2.54mm
- U7: renamed from U?; footprint (none) -> Package_DIP:DIP-20_W7.62mm_Socket
Changed lines of the file:
@@
 $Descr A4 11693 8268
 encoding utf-8
-Sheet 3 3
+Sheet 3 9
 Title ""
 Date ""
@@
 $EndDescr
 $Comp
-L Switch:SW_DIP_x08 SW?
+L Switch:SW_DIP_x08 SW4
 U 1 1 5B2C1F8A
 P 1250 1050
-F 0 "SW?" V 1296 620 50  0000 R CNN
+F 0 "SW4" V 1296 620 50  0000 R CNN
 F 1 "SW_DIP_x08" V 1205 620 50  0000 R CNN
-F 2 "" H 1250 1050 50  0001 C CNN
+F 2 "Button_Switch_THT:SW_DIP_SPSTx08_Slide_9.78x22.5mm_W7.62mm_P2.54mm" H 1250 1050 50  0001 C CNN
 F 3 "" H 1250 1050 50  0001 C CNN
 	1    1250 1050
@@
 $EndComp
 $Comp
-L power:VCC #PWR?
+L power:VCC #PWR0125
 U 1 1 5B2C21F5
 P 850 750
-F 0 "#PWR?" H 850 600 50  0001 C CNN
+F 0 "#PWR0125" H 850 600 50  0001 C CNN
 F 1 "VCC" H 867 923 50  0000 C CNN
 F 2 "" H 850 750 50  0001 C CNN
@@
 Connection ~ 1450 750
 $Comp
-L Device:R R?
+L Device:R R15
 U 1 1 5B2C25DC
 P 850 2700
-F 0 "R?" H 750 2850 50  0000 L CNN
+F 0 "R15" H 750 2850 50  0000 L CNN
 F 1 "100K" V 850 2600 50  0000 L CNN
-F 2 "" V 780 2700 50  0001 C CNN
+F 2 "Resistor_THT:R_Axial_DIN0207_L6.3mm_D2.5mm_P7.62mm_Horizontal" V 780 2700 50  0001 C CNN
 F 3 "~" H 850 2700 50  0001 C CNN
 	1    850  2700
@@
 $EndComp
 $Comp
-L Device:R R?
+L Device:R R16
 U 1 1 5B2C2BC6
 P 950 2700
-F 0 "R?" H 850 2850 50  0000 L CNN
+F 0 "R16" H 850 2850 50  0000 L CNN
 F 1 "100K" V 950 2600 50  0000 L CNN
-F 2 "" V 880 2700 50  0001 C CNN
+F 2 "Resistor_THT:R_Axial_DIN0207_L6.3mm_D2.5mm_P7.62mm_Horizontal" V 880 2700 50  0001 C CNN
 F 3 "~" H 950 2700 50  0001 C CNN
 	1    950  2700
@@
 $EndComp
 $Comp
-L Device:R R?
+L Device:R R17
 U 1 1 5B2C2C99
 P 1050 2700
-F 0 "R?" H 950 2850 50  0000 L CNN
+F 0 "R17" H 950 2850 50  0000 L CNN
 F 1 "100K" V 1050 2600 50  0000 L CNN
-F 2 "" V 980 2700 50  0001 C CNN
+F 2 "Resistor_THT:R_Axial_DIN0207_L6.3mm_D2.5mm_P7.62mm_Horizontal" V 980 2700 50  0001 C CNN
 F 3 "~" H 1050 2700 50  0001 C CNN
 	1    1050 2700
@@
 $EndComp
 $Comp
-L Device:R R?
+L Device:R R18
 U 1 1 5B2C2DA5
 P 1150 2700
-F 0 "R?" H 1050 2850 50  0000 L CNN
+F 0 "R18" H 1050 2850 50  0000 L CNN
 F 1 "100K" V 1150 2600 50  0000 L CNN
-F 2 "" V 1080 2700 50  0001 C CNN
+F 2 "Resistor_THT:R_Axial_DIN0207_L6.3mm_D2.5mm_P7.62mm_Horizontal" V 1080 2700 50  0001 C CNN
 F 3 "~" H 1150 2700 50  0001 C CNN
 	1    1150 2700
@@
 $EndComp
 $Comp
-L Device:R R?
+L Device:R R19
 U 1 1 5B2C2E95
 P 1250 2700
-F 0 "R?" H 1150 2850 50  0000 L CNN
+F 0 "R19" H 1150 2850 50  0000 L CNN
 F 1 "100K" V 1250 2600 50  0000 L CNN
-F 2 "" V 1180 2700 50  0001 C CNN
+F 2 "Resistor_THT:R_Axial_DIN0207_L6.3mm_D2.5mm_P7.62mm_Horizontal" V 1180 2700 50  0001 C CNN
 F 3 "~" H 1250 2700 50  0001 C CNN
 	1    1250 2700
@@
 $EndComp
 $Comp
-L Device:R R?
+L Device:R R20
 U 1 1 5B2C2FA7
 P 1350 2700
-F 0 "R?" H 1250 2850 50  0000 L CNN
+F 0 "R20" H 1250 2850 50  0000 L CNN
 F 1 "100K" V 1350 2600 50  0000 L CNN
-F 2 "" V 1280 2700 50  0001 C CNN
+F 2 "Resistor_THT:R_Axial_DIN0207_L6.3mm_D2.5mm_P7.62mm_Horizontal" V 1280 2700 50  0001 C CNN
 F 3 "~" H 1350 2700 50  0001 C CNN
 	1    1350 2700
@@
 $EndComp
 $Comp
-L Device:R R?
+L Device:R R21
 U 1 1 5B2C305F
 P 1450 2700
-F 0 "R?" H 1350 2850 50  0000 L CNN
+F 0 "R21" H 1350 2850 50  0000 L CNN
 F 1 "100K" V 1450 2600 50  0000 L CNN
-F 2 "" V 1380 2700 50  0001 C CNN
+F 2 "Resistor_THT:R_Axial_DIN0207_L6.3mm_D2.5mm_P7.62mm_Horizontal" V 1380 2700 50  0001 C CNN
 F 3 "~" H 1450 2700 50  0001 C CNN
 	1    1450 2700
@@
 $EndComp
 $Comp
-L Device:R R?
+L Device:R R22
 U 1 1 5B2C312F
 P 1550 2700
-F 0 "R?" H 1450 2850 50  0000 L CNN
+F 0 "R22" H 1450 2850 50  0000 L CNN
 F 1 "100K" V 1550 2600 50  0000 L CNN
-F 2 "" V 1480 2700 50  0001 C CNN
+F 2 "Resistor_THT:R_Axial_DIN0207_L6.3mm_D2.5mm_P7.62mm_Horizontal" V 1480 2700 50  0001 C CNN
 F 3 "~" H 1550 2700 50  0001 C CNN
 	1    1550 2700
@@
 $EndComp
 $Comp
-L 74xx:74HC245 U?
+L 74xx:74HC245 U7
 U 1 1 5B2C3561
 P 2200 1850
-F 0 "U?" H 2300 2500 50  0000 C CNN
+F 0 "U7" H 2300 2500 50  0000 C CNN
 F 1 "74HC245" H 2200 1550 50  0000 C CNN
-F 2 "" H 2200 1850 50  0001 C CNN
+F 2 "Package_DIP:DIP-20_W7.62mm_Socket" H 2200 1850 50  0001 C CNN
 F 3 "http://www.ti.com/lit/gpn/sn74HC245" H 2200 1850 50  0001 C CNN
 	1    2200 1850
@@
 $EndComp
 $Comp
-L power:VCC #PWR?
+L power:VCC #PWR0126
 U 1 1 5B2C3FAF
 P 2200 1050
-F 0 "#PWR?" H 2200 900 50  0001 C CNN
+F 0 "#PWR0126" H 2200 900 50  0001 C CNN
 F 1 "VCC" H 2217 1223 50  0000 C CNN
 F 2 "" H 2200 1050 50  0001 C CNN
@@
 $EndComp
 $Comp
-L power:GND #PWR?
+L power:GND #PWR0127
 U 1 1 5B2C4405
 P 2200 2650
-F 0 "#PWR?" H 2200 2400 50  0001 C CNN
+F 0 "#PWR0127" H 2200 2400 50  0001 C CNN
 F 1 "GND" H 2205 2477 50  0000 C CNN
 F 2 "" H 2200 2650 50  0001 C CNN
@@
 $EndComp
 $Comp
-L power:GND #PWR?
+L power:GND #PWR0128
 U 1 1 5B2CAE54
 P 850 2850
-F 0 "#PWR?" H 850 2600 50  0001 C CNN
+F 0 "#PWR0128" H 850 2600 50  0001 C CNN
 F 1 "GND" H 855 2677 50  0000 C CNN
 F 2 "" H 850 2850 50  0001 C CNN
@@
 Connection ~ 850  2050
 $Comp
-L power:VCC #PWR?
+L power:VCC #PWR0129
 U 1 1 5B2DCAC9
 P 1700 2250
-F 0 "#PWR?" H 1700 2100 50  0001 C CNN
+F 0 "#PWR0129" H 1700 2100 50  0001 C CNN
 F 1 "VCC" H 1717 2423 50  0000 C CNN
 F 2 "" H 1700 2250 50  0001 C CNN

Commit message: Schematic for kernel and user stack pointers.
Connections:
- net labels added: ~OUT
- net labels removed: OUT
Changed lines of the file:
@@
 $Descr A4 11693 8268
 encoding utf-8
-Sheet 3 17
+Sheet 3 19
 Title ""
 Date ""
@@
 $EndComp
 Text HLabel 1700 2350 0    50   Input ~ 0
-OUT
+~OUT
 Text HLabel 2700 1350 2    50   Input ~ 0
 O0
