File: kicad/register_with_bus_transceiver.sch (KiCad schematic (older format))
At the start: 4 parts, among them U8 74HCT574, U9 74HC245

Commit message: Start program counter. Write down design notes.
Changed lines of the file:
@@
 $Descr A4 11693 8268
 encoding utf-8
-Sheet 11 14
+Sheet 10 17
 Title ""
 Date ""
@@
 AR Path="/5AFD5CE2/5AFCCD08/5AFCD0D6" Ref="U8"  Part="1"
 AR Path="/5AFD5CE2/5AFD336A/5AFCD0D6" Ref="U10"  Part="1"
-F 0 "U10" H 1850 2650 50  0000 C CNN
+F 0 "U8" H 1850 2650 50  0000 C CNN
 F 1 "74HCT574" H 1750 1650 50  0000 C CNN
 F 2 "Package_DIP:DIP-20_W7.62mm_Socket" H 1750 1950 50  0001 C CNN
@@
 AR Path="/5AFD5CE2/5AFCCD08/5AFCD0DD" Ref="#PWR024"  Part="1"
 AR Path="/5AFD5CE2/5AFD336A/5AFCD0DD" Ref="#PWR032"  Part="1"
-F 0 "#PWR032" H 1750 2500 50  0001 C CNN
+F 0 "#PWR024" H 1750 2500 50  0001 C CNN
 F 1 "GND" H 1755 2577 50  0000 C CNN
 F 2 "" H 1750 2750 50  0001 C CNN
@@
 AR Path="/5AFD5CE2/5AFCCD08/5AFCD0E3" Ref="#PWR023"  Part="1"
 AR Path="/5AFD5CE2/5AFD336A/5AFCD0E3" Ref="#PWR031"  Part="1"
-F 0 "#PWR031" H 1750 1000 50  0001 C CNN
+F 0 "#PWR023" H 1750 1000 50  0001 C CNN
 F 1 "VCC" H 1767 1323 50  0000 C CNN
 F 2 "" H 1750 1150 50  0001 C CNN
@@
 AR Path="/5AFD5CE2/5AFCCD08/5AFCD0FB" Ref="C20"  Part="1"
 AR Path="/5AFD5CE2/5AFD336A/5AFCD0FB" Ref="C22"  Part="1"
-F 0 "C22" H 792 1896 50  0000 L CNN
+F 0 "C20" H 792 1896 50  0000 L CNN
 F 1 "0.1uF" H 792 1805 50  0000 L CNN
 F 2 "Capacitor_THT:C_Disc_D3.0mm_W2.0mm_P2.50mm" H 700 1850 50  0001 C CNN
@@
 AR Path="/5AFD5CE2/5AFCCD08/5AFCDA3B" Ref="U9"  Part="1"
 AR Path="/5AFD5CE2/5AFD336A/5AFCDA3B" Ref="U11"  Part="1"
-F 0 "U11" H 3950 2700 50  0000 C CNN
+F 0 "U9" H 3950 2700 50  0000 C CNN
 F 1 "74HC245" H 3900 1700 50  0000 C CNN
 F 2 "Package_DIP:DIP-20_W7.62mm_Socket" H 3850 2000 50  0001 C CNN
@@
 AR Path="/5AFD5CE2/5AFCCD08/5AFCDF58" Ref="#PWR016"  Part="1"
 AR Path="/5AFD5CE2/5AFD336A/5AFCDF58" Ref="#PWR030"  Part="1"
-F 0 "#PWR030" H 1250 2200 50  0001 C CNN
+F 0 "#PWR016" H 1250 2200 50  0001 C CNN
 F 1 "GND" H 1255 2277 50  0000 C CNN
 F 2 "" H 1250 2450 50  0001 C CNN
@@
 AR Path="/5AFD5CE2/5AFCCD08/5AFCF275" Ref="#PWR029"  Part="1"
 AR Path="/5AFD5CE2/5AFD336A/5AFCF275" Ref="#PWR037"  Part="1"
-F 0 "#PWR037" H 3850 2550 50  0001 C CNN
+F 0 "#PWR029" H 3850 2550 50  0001 C CNN
 F 1 "GND" H 3855 2627 50  0000 C CNN
 F 2 "" H 3850 2800 50  0001 C CNN
@@
 AR Path="/5AFD5CE2/5AFCCD08/5AFCF63F" Ref="C21"  Part="1"
 AR Path="/5AFD5CE2/5AFD336A/5AFCF63F" Ref="C23"  Part="1"
-F 0 "C23" H 2892 1946 50  0000 L CNN
+F 0 "C21" H 2892 1946 50  0000 L CNN
 F 1 "0.1uF" H 2892 1855 50  0000 L CNN
 F 2 "Capacitor_THT:C_Disc_D3.0mm_W2.0mm_P2.50mm" H 2800 1900 50  0001 C CNN
@@
 AR Path="/5AFD5CE2/5AFCCD08/5AFCFAAC" Ref="#PWR026"  Part="1"
 AR Path="/5AFD5CE2/5AFD336A/5AFCFAAC" Ref="#PWR036"  Part="1"
-F 0 "#PWR036" H 3850 1050 50  0001 C CNN
+F 0 "#PWR026" H 3850 1050 50  0001 C CNN
 F 1 "VCC" H 3867 1373 50  0000 C CNN
 F 2 "" H 3850 1200 50  0001 C CNN
@@
 AR Path="/5AFD5CE2/5AFCCD08/5AFCFCC3" Ref="#PWR025"  Part="1"
 AR Path="/5AFD5CE2/5AFD336A/5AFCFCC3" Ref="#PWR035"  Part="1"
-F 0 "#PWR035" H 3350 2250 50  0001 C CNN
+F 0 "#PWR025" H 3350 2250 50  0001 C CNN
 F 1 "VCC" H 3367 2573 50  0000 C CNN
 F 2 "" H 3350 2400 50  0001 C CNN

Commit message: Add SC register and program counter.
Changed lines of the file:
@@
 AR Path="/5AFD5CE2/5AFCCD08/5AFCD0D6" Ref="U8"  Part="1"
 AR Path="/5AFD5CE2/5AFD336A/5AFCD0D6" Ref="U10"  Part="1"
-F 0 "U8" H 1850 2650 50  0000 C CNN
+F 0 "U10" H 1850 2650 50  0000 C CNN
 F 1 "74HCT574" H 1750 1650 50  0000 C CNN
 F 2 "Package_DIP:DIP-20_W7.62mm_Socket" H 1750 1950 50  0001 C CNN
@@
 AR Path="/5AFD5CE2/5AFCCD08/5AFCD0DD" Ref="#PWR024"  Part="1"
 AR Path="/5AFD5CE2/5AFD336A/5AFCD0DD" Ref="#PWR032"  Part="1"
-F 0 "#PWR024" H 1750 2500 50  0001 C CNN
+F 0 "#PWR032" H 1750 2500 50  0001 C CNN
 F 1 "GND" H 1755 2577 50  0000 C CNN
 F 2 "" H 1750 2750 50  0001 C CNN
@@
 AR Path="/5AFD5CE2/5AFCCD08/5AFCD0E3" Ref="#PWR023"  Part="1"
 AR Path="/5AFD5CE2/5AFD336A/5AFCD0E3" Ref="#PWR031"  Part="1"
-F 0 "#PWR023" H 1750 1000 50  0001 C CNN
+F 0 "#PWR031" H 1750 1000 50  0001 C CNN
 F 1 "VCC" H 1767 1323 50  0000 C CNN
 F 2 "" H 1750 1150 50  0001 C CNN
@@
 AR Path="/5AFD5CE2/5AFCCD08/5AFCD0FB" Ref="C20"  Part="1"
 AR Path="/5AFD5CE2/5AFD336A/5AFCD0FB" Ref="C22"  Part="1"
-F 0 "C20" H 792 1896 50  0000 L CNN
+F 0 "C22" H 792 1896 50  0000 L CNN
 F 1 "0.1uF" H 792 1805 50  0000 L CNN
 F 2 "Capacitor_THT:C_Disc_D3.0mm_W2.0mm_P2.50mm" H 700 1850 50  0001 C CNN
@@
 AR Path="/5AFD5CE2/5AFCCD08/5AFCDA3B" Ref="U9"  Part="1"
 AR Path="/5AFD5CE2/5AFD336A/5AFCDA3B" Ref="U11"  Part="1"
-F 0 "U9" H 3950 2700 50  0000 C CNN
+F 0 "U11" H 3950 2700 50  0000 C CNN
 F 1 "74HC245" H 3900 1700 50  0000 C CNN
 F 2 "Package_DIP:DIP-20_W7.62mm_Socket" H 3850 2000 50  0001 C CNN
@@
 AR Path="/5AFD5CE2/5AFCCD08/5AFCDF58" Ref="#PWR016"  Part="1"
 AR Path="/5AFD5CE2/5AFD336A/5AFCDF58" Ref="#PWR030"  Part="1"
-F 0 "#PWR016" H 1250 2200 50  0001 C CNN
+F 0 "#PWR030" H 1250 2200 50  0001 C CNN
 F 1 "GND" H 1255 2277 50  0000 C CNN
 F 2 "" H 1250 2450 50  0001 C CNN
@@
 AR Path="/5AFD5CE2/5AFCCD08/5AFCF275" Ref="#PWR029"  Part="1"
 AR Path="/5AFD5CE2/5AFD336A/5AFCF275" Ref="#PWR037"  Part="1"
-F 0 "#PWR029" H 3850 2550 50  0001 C CNN
+F 0 "#PWR037" H 3850 2550 50  0001 C CNN
 F 1 "GND" H 3855 2627 50  0000 C CNN
 F 2 "" H 3850 2800 50  0001 C CNN
@@
 AR Path="/5AFD5CE2/5AFCCD08/5AFCF63F" Ref="C21"  Part="1"
 AR Path="/5AFD5CE2/5AFD336A/5AFCF63F" Ref="C23"  Part="1"
-F 0 "C21" H 2892 1946 50  0000 L CNN
+F 0 "C23" H 2892 1946 50  0000 L CNN
 F 1 "0.1uF" H 2892 1855 50  0000 L CNN
 F 2 "Capacitor_THT:C_Disc_D3.0mm_W2.0mm_P2.50mm" H 2800 1900 50  0001 C CNN
@@
 AR Path="/5AFD5CE2/5AFCCD08/5AFCFAAC" Ref="#PWR026"  Part="1"
 AR Path="/5AFD5CE2/5AFD336A/5AFCFAAC" Ref="#PWR036"  Part="1"
-F 0 "#PWR026" H 3850 1050 50  0001 C CNN
+F 0 "#PWR036" H 3850 1050 50  0001 C CNN
 F 1 "VCC" H 3867 1373 50  0000 C CNN
 F 2 "" H 3850 1200 50  0001 C CNN
@@
 AR Path="/5AFD5CE2/5AFCCD08/5AFCFCC3" Ref="#PWR025"  Part="1"
 AR Path="/5AFD5CE2/5AFD336A/5AFCFCC3" Ref="#PWR035"  Part="1"
-F 0 "#PWR025" H 3350 2250 50  0001 C CNN
+F 0 "#PWR035" H 3350 2250 50  0001 C CNN
 F 1 "VCC" H 3367 2573 50  0000 C CNN
 F 2 "" H 3350 2400 50  0001 C CNN

Commit message: Schematic for kernel and user stack pointers.
Connections:
- net labels added: ~REG_OUT
- net labels removed: REG_OUT
Changed lines of the file:
@@
 $Descr A4 11693 8268
 encoding utf-8
-Sheet 10 17
+Sheet 10 19
 Title ""
 Date ""
@@
 I7
 Text HLabel 3350 2500 0    50   Input ~ 0
-REG_OUT
+~REG_OUT
 Text HLabel 2250 1450 2    50   Input ~ 0
 O0

Commit message: Finish MMU schematic.
Parts:
- renumbered C20 to C19, C21 to C20
Changed lines of the file:
@@
 $Descr A4 11693 8268
 encoding utf-8
-Sheet 10 23
+Sheet 9 23
 Title ""
 Date ""
@@
 AR Path="/5AFD5CE2/5AFD86BE/5AFCD0D6" Ref="U?"  Part="1"
 AR Path="/5AFD5CE2/5AFCCD08/5AFCD0D6" Ref="U8"  Part="1"
-AR Path="/5AFD5CE2/5AFD336A/5AFCD0D6" Ref="U10"  Part="1"
-F 0 "U10" H 1850 2650 50  0000 C CNN
+AR Path="/5AFD5CE2/5AFD336A/5AFCD0D6" Ref="U18"  Part="1"
+AR Path="/5AFD5CE2/5B0AB8A7/5AFCD0D6" Ref="U10"  Part="1"
+F 0 "U18" H 1850 2650 50  0000 C CNN
 F 1 "74HCT574" H 1750 1650 50  0000 C CNN
 F 2 "Package_DIP:DIP-20_W7.62mm_Socket" H 1750 1950 50  0001 C CNN
@@
 $EndComp
 $Comp
-L power:GND #PWR024
+L power:GND #PWR0285
 U 1 1 5AFCD0DD
 P 1750 2750
-AR Path="/5AFD5CE2/5AFCCD08/5AFCD0DD" Ref="#PWR024"  Part="1"
-AR Path="/5AFD5CE2/5AFD336A/5AFCD0DD" Ref="#PWR032"  Part="1"
-F 0 "#PWR032" H 1750 2500 50  0001 C CNN
+AR Path="/5AFD5CE2/5AFCCD08/5AFCD0DD" Ref="#PWR0285"  Part="1"
+AR Path="/5AFD5CE2/5B0AB8A7/5AFCD0DD" Ref="#PWR0321"  Part="1"
+AR Path="/5AFD5CE2/5AFD336A/5AFCD0DD" Ref="#PWR0327"  Part="1"
+F 0 "#PWR0327" H 1750 2500 50  0001 C CNN
 F 1 "GND" H 1755 2577 50  0000 C CNN
 F 2 "" H 1750 2750 50  0001 C CNN
@@
 $EndComp
 $Comp
-L power:VCC #PWR023
+L power:VCC #PWR0286
 U 1 1 5AFCD0E3
 P 1750 1150
-AR Path="/5AFD5CE2/5AFCCD08/5AFCD0E3" Ref="#PWR023"  Part="1"
-AR Path="/5AFD5CE2/5AFD336A/5AFCD0E3" Ref="#PWR031"  Part="1"
-F 0 "#PWR031" H 1750 1000 50  0001 C CNN
+AR Path="/5AFD5CE2/5AFCCD08/5AFCD0E3" Ref="#PWR0286"  Part="1"
+AR Path="/5AFD5CE2/5B0AB8A7/5AFCD0E3" Ref="#PWR0322"  Part="1"
+AR Path="/5AFD5CE2/5AFD336A/5AFCD0E3" Ref="#PWR0328"  Part="1"
+F 0 "#PWR0328" H 1750 1000 50  0001 C CNN
 F 1 "VCC" H 1767 1323 50  0000 C CNN
 F 2 "" H 1750 1150 50  0001 C CNN
@@
 O7
 $Comp
-L Device:C_Small C20
+L Device:C_Small C19
 U 1 1 5AFCD0FB
 P 700 1850
-AR Path="/5AFD5CE2/5AFCCD08/5AFCD0FB" Ref="C20"  Part="1"
-AR Path="/5AFD5CE2/5AFD336A/5AFCD0FB" Ref="C22"  Part="1"
-F 0 "C22" H 792 1896 50  0000 L CNN
+AR Path="/5AFD5CE2/5AFCCD08/5AFCD0FB" Ref="C19"  Part="1"
+AR Path="/5AFD5CE2/5B0AB8A7/5AFCD0FB" Ref="C21"  Part="1"
+AR Path="/5AFD5CE2/5AFD336A/5AFCD0FB" Ref="C23"  Part="1"
+F 0 "C23" H 792 1896 50  0000 L CNN
 F 1 "0.1uF" H 792 1805 50  0000 L CNN
 F 2 "Capacitor_THT:C_Disc_D3.0mm_W2.0mm_P2.50mm" H 700 1850 50  0001 C CNN
@@
 P 3850 2000
 AR Path="/5AFD5CE2/5AFCCD08/5AFCDA3B" Ref="U9"  Part="1"
-AR Path="/5AFD5CE2/5AFD336A/5AFCDA3B" Ref="U11"  Part="1"
-F 0 "U11" H 3950 2700 50  0000 C CNN
+AR Path="/5AFD5CE2/5AFD336A/5AFCDA3B" Ref="U83"  Part="1"
+AR Path="/5AFD5CE2/5B0AB8A7/5AFCDA3B" Ref="U11"  Part="1"
+F 0 "U83" H 3950 2700 50  0000 C CNN
 F 1 "74HC245" H 3900 1700 50  0000 C CNN
 F 2 "Package_DIP:DIP-20_W7.62mm_Socket" H 3850 2000 50  0001 C CNN
@@
 $EndComp
 $Comp
-L power:GND #PWR016
+L power:GND #PWR0317
 U 1 1 5AFCDF58
 P 1250 2450
-AR Path="/5AFD5CE2/5AFCCD08/5AFCDF58" Ref="#PWR016"  Part="1"
-AR Path="/5AFD5CE2/5AFD336A/5AFCDF58" Ref="#PWR030"  Part="1"
-F 0 "#PWR030" H 1250 2200 50  0001 C CNN
+AR Path="/5AFD5CE2/5AFCCD08/5AFCDF58" Ref="#PWR0317"  Part="1"
+AR Path="/5AFD5CE2/5B0AB8A7/5AFCDF58" Ref="#PWR0323"  Part="1"
+AR Path="/5AFD5CE2/5AFD336A/5AFCDF58" Ref="#PWR0329"  Part="1"
+F 0 "#PWR0329" H 1250 2200 50  0001 C CNN
 F 1 "GND" H 1255 2277 50  0000 C CNN
 F 2 "" H 1250 2450 50  0001 C CNN
@@
 BUS7
 $Comp
-L power:GND #PWR029
+L power:GND #PWR0318
 U 1 1 5AFCF275
 P 3850 2800
-AR Path="/5AFD5CE2/5AFCCD08/5AFCF275" Ref="#PWR029"  Part="1"
-AR Path="/5AFD5CE2/5AFD336A/5AFCF275" Ref="#PWR037"  Part="1"
-F 0 "#PWR037" H 3850 2550 50  0001 C CNN
+AR Path="/5AFD5CE2/5AFCCD08/5AFCF275" Ref="#PWR0318"  Part="1"
+AR Path="/5AFD5CE2/5B0AB8A7/5AFCF275" Ref="#PWR0324"  Part="1"
+AR Path="/5AFD5CE2/5AFD336A/5AFCF275" Ref="#PWR0330"  Part="1"
+F 0 "#PWR0330" H 3850 2550 50  0001 C CNN
 F 1 "GND" H 3855 2627 50  0000 C CNN
 F 2 "" H 3850 2800 50  0001 C CNN
@@
 $EndComp
 $Comp
-L Device:C_Small C21
+L Device:C_Small C20
 U 1 1 5AFCF63F
 P 2800 1900
-AR Path="/5AFD5CE2/5AFCCD08/5AFCF63F" Ref="C21"  Part="1"
-AR Path="/5AFD5CE2/5AFD336A/5AFCF63F" Ref="C23"  Part="1"
-F 0 "C23" H 2892 1946 50  0000 L CNN
+AR Path="/5AFD5CE2/5AFCCD08/5AFCF63F" Ref="C20"  Part="1"
+AR Path="/5AFD5CE2/5B0AB8A7/5AFCF63F" Ref="C22"  Part="1"
+AR Path="/5AFD5CE2/5AFD336A/5AFCF63F" Ref="C90"  Part="1"
+F 0 "C90" H 2892 1946 50  0000 L CNN
 F 1 "0.1uF" H 2892 1855 50  0000 L CNN
 F 2 "Capacitor_THT:C_Disc_D3.0mm_W2.0mm_P2.50mm" H 2800 1900 50  0001 C CNN
@@
 Connection ~ 3850 2800
 $Comp
-L power:VCC #PWR026
+L power:VCC #PWR0319
 U 1 1 5AFCFAAC
 P 3850 1200
-AR Path="/5AFD5CE2/5AFCCD08/5AFCFAAC" Ref="#PWR026"  Part="1"
-AR Path="/5AFD5CE2/5AFD336A/5AFCFAAC" Ref="#PWR036"  Part="1"
-F 0 "#PWR036" H 3850 1050 50  0001 C CNN
+AR Path="/5AFD5CE2/5AFCCD08/5AFCFAAC" Ref="#PWR0319"  Part="1"
+AR Path="/5AFD5CE2/5B0AB8A7/5AFCFAAC" Ref="#PWR0325"  Part="1"
+AR Path="/5AFD5CE2/5AFD336A/5AFCFAAC" Ref="#PWR0331"  Part="1"
+F 0 "#PWR0331" H 3850 1050 50  0001 C CNN
 F 1 "VCC" H 3867 1373 50  0000 C CNN
 F 2 "" H 3850 1200 50  0001 C CNN
@@
 Connection ~ 3850 1200
 $Comp
-L power:VCC #PWR025
+L power:VCC #PWR0320
 U 1 1 5AFCFCC3
 P 3350 2400
-AR Path="/5AFD5CE2/5AFCCD08/5AFCFCC3" Ref="#PWR025"  Part="1"
-AR Path="/5AFD5CE2/5AFD336A/5AFCFCC3" Ref="#PWR035"  Part="1"
-F 0 "#PWR035" H 3350 2250 50  0001 C CNN
+AR Path="/5AFD5CE2/5AFCCD08/5AFCFCC3" Ref="#PWR0320"  Part="1"
+AR Path="/5AFD5CE2/5B0AB8A7/5AFCFCC3" Ref="#PWR0326"  Part="1"
+AR Path="/5AFD5CE2/5AFD336A/5AFCFCC3" Ref="#PWR0332"  Part="1"
+F 0 "#PWR0332" H 3350 2250 50  0001 C CNN
 F 1 "VCC" H 3367 2573 50  0000 C CNN
 F 2 "" H 3350 2400 50  0001 C CNN
