File: kicad/mmu.sch (KiCad schematic (older format))
At the start: 19 parts, among them U70 74LS154, U71 SST39SF040, U72 628128, U73 628128, U74 628128, U75 628128, U76 628128, U77 628128, U78 628128, U79 628128

Commit message: Finish MMU schematic.
Parts:
- added C91, C92, C93, C94: 0.1uF, Capacitor_THT:C_Disc_D3.0mm_W2.0mm_P2.50mm, symbol Device:C_Small
- added U84: 628128, Package_DIP:DIP-32_W15.24mm_Socket, symbol Memory_RAM:628128
- added U85: 74LS153, Package_DIP:DIP-16_W7.62mm_Socket, symbol 74xx:74LS153
- added U86: 74HC245, Package_DIP:DIP-20_W7.62mm_Socket, symbol 74xx:74HC245
- C78, C79, C80, C81, C82, C83, C84, C85, C86: value C_Small -> 0.1uF
Connections:
- net labels added: MMU_READ_FAULT, MMU_WRITE_FAULT, READ0, READ1, READ2, READ3, TASK0, TASK1, TASK2, TASK3, TASK4, TASK5, TASK6, TASK7, WRITE0, WRITE1, WRITE2, WRITE3, ~MMU_CONTROL_IN, ~MMU_CONTROL_OUT
- wire segments 0 -> 11
Other:
- note added: "M20 reads from memory \nmapped eeprom instead."
- note added: "Use 4-16 line decoder to select\nwhich memory chip to use."
- note removed: "TODO: Check VCC and GND are connected for hidden pins on sram, eeprom"
- note removed: "TODO: Need to make task register have a bus transceiver to plug into memory protection hardware."

Commit message: Layout MMU.
Changed lines of the file:
@@
 Text HLabel -750 4600 2    50   Input ~ 0
 MMU_WRITE_FAULT
+Text HLabel 900  1050 0    50   Input ~ 0
+BUS0
+Text HLabel 900  1150 0    50   Input ~ 0
+BUS1
+Text HLabel 900  1250 0    50   Input ~ 0
+BUS2
+Text HLabel 900  1350 0    50   Input ~ 0
+BUS3
+Text HLabel 900  1450 0    50   Input ~ 0
+BUS4
+Text HLabel 900  1550 0    50   Input ~ 0
+BUS5
+Text HLabel 900  1650 0    50   Input ~ 0
+BUS6
+Text HLabel 900  1750 0    50   Input ~ 0
+BUS7
+Text HLabel 2050 1050 0    50   Input ~ 0
+BUS0
+Text HLabel 2050 1150 0    50   Input ~ 0
+BUS1
+Text HLabel 2050 1250 0    50   Input ~ 0
+BUS2
+Text HLabel 2050 1350 0    50   Input ~ 0
+BUS3
+Text HLabel 2050 1450 0    50   Input ~ 0
+BUS4
+Text HLabel 2050 1550 0    50   Input ~ 0
+BUS5
+Text HLabel 2050 1650 0    50   Input ~ 0
+BUS6
+Text HLabel 2050 1750 0    50   Input ~ 0
+BUS7
+Text HLabel 3300 1050 0    50   Input ~ 0
+BUS0
+Text HLabel 3300 1150 0    50   Input ~ 0
+BUS1
+Text HLabel 3300 1250 0    50   Input ~ 0
+BUS2
+Text HLabel 3300 1350 0    50   Input ~ 0
+BUS3
+Text HLabel 3300 1450 0    50   Input ~ 0
+BUS4
+Text HLabel 3300 1550 0    50   Input ~ 0
+BUS5
+Text HLabel 3300 1650 0    50   Input ~ 0
+BUS6
+Text HLabel 3300 1750 0    50   Input ~ 0
+BUS7
 $EndSCHEMATC

Commit message: Annotate
Other:
- moved on the sheet: U86

Commit message: Start connecting up control logic.
Connections:
- net labels added: MMU0_IN, MMU1_IN, MMU2_IN
Changed lines of the file:
@@
 Text HLabel 8000 1750 0    50   Input ~ 0
 BUS7
+$Comp
+L power:GND #PWR?
+U 1 1 5B1F8EE4
+P 5600 1950
+F 0 "#PWR?" H 5600 1700 50  0001 C CNN
+F 1 "GND" H 5605 1777 50  0000 C CNN
+F 2 "" H 5600 1950 50  0001 C CNN
+F 3 "" H 5600 1950 50  0001 C CNN
+	1    5600 1950
+	0    1    1    0
+$EndComp
+$Comp
+L power:GND #PWR?
+U 1 1 5B1F8F3D
+P 6750 1950
+F 0 "#PWR?" H 6750 1700 50  0001 C CNN
+F 1 "GND" H 6755 1777 50  0000 C CNN
+F 2 "" H 6750 1950 50  0001 C CNN
+F 3 "" H 6750 1950 50  0001 C CNN
+	1    6750 1950
+	0    1    1    0
+$EndComp
+$Comp
+L power:GND #PWR?
+U 1 1 5B1F902C
+P 8000 1950
+F 0 "#PWR?" H 8000 1700 50  0001 C CNN
+F 1 "GND" H 8005 1777 50  0000 C CNN
+F 2 "" H 8000 1950 50  0001 C CNN
+F 3 "" H 8000 1950 50  0001 C CNN
+	1    8000 1950
+	0    1    1    0
+$EndComp
+Text HLabel 5600 2050 0    50   Input ~ 0
+MMU0_IN
+Text HLabel 6750 2050 0    50   Input ~ 0
+MMU1_IN
+Text HLabel 8000 2050 0    50   Input ~ 0
+MMU2_IN
 $EndSCHEMATC
