File: kicad/stack_register.sch (KiCad schematic (older format))
At the start: 31 parts

Commit message: Layout user and kernel stack pointers.
Parts:
- added C76: 0.1uF, Capacitor_THT:C_Disc_D3.0mm_W2.0mm_P2.50mm, symbol Device:C_Small
- gave numbers to parts that had none: 21
