File: kicad/cpu.sch (KiCad schematic (older format))
At the start: 7 parts, among them J1 Conn_01x05, SW3 SW_DPST

Commit message: Small progress.
Connections:
- net labels added: ~CLK
Changed lines of the file:
@@
 F2 "CLK" I R 1650 1050 50
 F3 "~RESET" I L 1000 1050 50
+F4 "~CLK" I R 1650 1200 50
 $EndSheet
 $Comp
@@
 F1 "control_logic.sch" 50
 $EndSheet
+Text Label 1650 1200 0    50   ~ 0
+~CLK
 $EndSCHEMATC

Commit message: Progress on control logic. Micro-op counter. Opcode register.
Connections:
- net labels added: MMU_READ_FAULT, MMU_WRITE_FAULT
Changed lines of the file:
@@
 $Descr A4 11693 8268
 encoding utf-8
-Sheet 1 34
+Sheet 1 36
 Title ""
 Date ""
@@
 Text Label 1650 1200 0    50   ~ 0
 ~CLK
+Text Label 7900 2800 0    50   ~ 0
+MMU_READ_FAULT
+Text Label 7900 2900 0    50   ~ 0
+MMU_WRITE_FAULT
 $EndSCHEMATC

Commit message: Control logic progress.
Connections:
- net labels added: INT0, INT1, INT2, INT3, INT4, INT5, INT6, INT7, INT_IN_CLK, ~INT_OUT
Changed lines of the file:
@@
 $Descr A4 11693 8268
 encoding utf-8
-Sheet 1 36
+Sheet 1 40
 Title ""
 Date ""
@@
 Text Label 7900 2900 0    50   ~ 0
 MMU_WRITE_FAULT
+$Sheet
+S 9200 3900 750  1750
+U 5B0FEA60
+F0 "Interrupt Register" 50
+F1 "register_with_bus_transceiver.sch" 50
+F2 "REG_IN" I L 9200 5550 50
+F3 "I0" I L 9200 4000 50
+F4 "I1" I L 9200 4100 50
+F5 "I2" I L 9200 4200 50
+F6 "I3" I L 9200 4300 50
+F7 "I4" I L 9200 4400 50
+F8 "I5" I L 9200 4500 50
+F9 "I6" I L 9200 4600 50
+F10 "I7" I L 9200 4700 50
+F11 "~REG_OUT" I L 9200 5450 50
+F12 "O0" I R 9950 4000 50
+F13 "O1" I R 9950 4100 50
+F14 "O2" I R 9950 4200 50
+F15 "O3" I R 9950 4300 50
+F16 "O4" I R 9950 4400 50
+F17 "O5" I R 9950 4500 50
+F18 "O6" I R 9950 4600 50
+F19 "O7" I R 9950 4700 50
+F20 "BUS0" I R 9950 4800 50
+F21 "BUS1" I R 9950 4900 50
+F22 "BUS2" I R 9950 5000 50
+F23 "BUS3" I R 9950 5100 50
+F24 "BUS4" I R 9950 5200 50
+F25 "BUS5" I R 9950 5300 50
+F26 "BUS6" I R 9950 5400 50
+F27 "BUS7" I R 9950 5500 50
+$EndSheet
+Text Label 9200 4000 2    50   ~ 0
+BUS0
+Text Label 9200 4100 2    50   ~ 0
+BUS1
+Text Label 9200 4200 2    50   ~ 0
+BUS2
+Text Label 9200 4300 2    50   ~ 0
+BUS3
+Text Label 9200 4400 2    50   ~ 0
+BUS4
+Text Label 9200 4500 2    50   ~ 0
+BUS5
+Text Label 9200 4600 2    50   ~ 0
+BUS6
+Text Label 9200 4700 2    50   ~ 0
+BUS7
+Text Label 9200 5450 2    50   ~ 0
+~INT_OUT
+Text Label 9200 5550 2    50   ~ 0
+INT_IN_CLK
+Text Label 9950 4000 0    50   ~ 0
+INT0
+Text Label 9950 4100 0    50   ~ 0
+INT1
+Text Label 9950 4200 0    50   ~ 0
+INT2
+Text Label 9950 4300 0    50   ~ 0
+INT3
+Text Label 9950 4400 0    50   ~ 0
+INT4
+Text Label 9950 4500 0    50   ~ 0
+INT5
+Text Label 9950 4600 0    50   ~ 0
+INT6
+Text Label 9950 4700 0    50   ~ 0
+INT7
+Text Label 9950 4800 0    50   ~ 0
+BUS0
+Text Label 9950 4900 0    50   ~ 0
+BUS1
+Text Label 9950 5000 0    50   ~ 0
+BUS2
+Text Label 9950 5100 0    50   ~ 0
+BUS3
+Text Label 9950 5200 0    50   ~ 0
+BUS4
+Text Label 9950 5300 0    50   ~ 0
+BUS5
+Text Label 9950 5400 0    50   ~ 0
+BUS6
+Text Label 9950 5500 0    50   ~ 0
+BUS7
 $EndSCHEMATC

Commit message: Control logic progress.
Connections:
- net labels added: INT0_LATCH, INT1_LATCH, INT2_LATCH, INT3_LATCH, INT4_LATCH, INT5_LATCH, INT6_LATCH, INT7_LATCH

Commit message: Annotate
Changed lines of the file:
@@
 F78 "INT6_LATCH" I L 1850 4350 50
 F79 "INT7_LATCH" I L 1850 4450 50
+F80 "INTERRUPT_ENABLE_FLAG" I L 1850 4550 50
 $EndSheet
 Text Label 1650 1200 0    50   ~ 0

Commit message: Start connecting up control logic.
Connections:
- net labels added: ALU_FLAG_SET_CLK, A_IN_CLK, B_IN_CLK, DISP_IN_CLK, INT0_IN_CLK, INT1_IN_CLK, INT2_IN_CLK, INT3_IN_CLK, INT4_IN_CLK, INT5_IN_CLK, INT6_IN_CLK, INT7_IN_CLK, K0_IN_CLK, K1_IN_CLK, K2_IN_CLK, KSP_DEC_CLK, KSP_INC_CLK, M0_IN_CLK, M1_IN_CLK, M2_IN_CLK, MLU_SEL0, MLU_SEL1, MLU_SEL2, MMU0_IN_CLK, MMU1_IN_CLK, MMU2_IN_CLK, MMU_CONTROL_IN_CLK, MMU_IN_CLK, PC0_IN_CLK, PC1_IN_CLK, PC2_IN_CLK, PC_INC_CLK, S0_IN_CLK, S1_IN_CLK, S2_IN_CLK, SP_DEC_CLK, SP_INC_CLK, TASK_IN_CLK, ~A_OUT_NCLK, ~B_OUT_NCLK, ~INTERRUPT_OUT_NCLK, ~K0_OUT_NCLK, ~K1_OUT_NCLK, ~K2_OUT_NCLK, ~M0_OUT_NCLK, ~M1_OUT_NCLK, ~M2_OUT_NCLK, ~MLU_OUT_NCLK, ~MMU_CONTROL_OUT_NCLK, ~MMU_OUT_NCLK, ~PC0_OUT_NCLK, ~PC1_OUT_NCLK, ~PC2_OUT_NCLK, ~RESET_NCLK, ~RESET_UOP_COUNT_NCLK, ~S0_OUT_NCLK, ~S1_OUT_NCLK, ~S2_OUT_NCLK, ~SET_INT_ENABLE_SYNC, ~STATUS_OUT_NCLK, ~SUB_NCLK, ~SUM_OUT_NCLK, ~TASK_OUT_NCLK, ~UNSET_INT_ENABLE_SYNC

Commit message: Control logic progress.
Connections:
- net labels added: CARRY, INTERRUPT_ENABLE_FLAG, SUB_NCLK, ZERO, ~K0_IN_CLK, ~K1_IN_CLK, ~K2_IN_CLK, ~PC0_IN_NCLK, ~PC1_IN_NCLK, ~PC2_IN_NCLK, ~S0_IN_CLK, ~S1_IN_CLK, ~S2_IN_CLK
- net labels removed: K0_IN_CLK, K1_IN_CLK, K2_IN_CLK, PC0_IN_CLK, PC1_IN_CLK, PC2_IN_CLK, S0_IN_CLK, S1_IN_CLK, S2_IN_CLK, ~SUB_NCLK
Other:
- note added: "TODO: output these onto the bus"
- note added: "TODO: why is PC_INC, etc clocked?"

Commit message: Fix PC INC, SP, KSP inc/dec.
Connections:
- net labels added: PC_INC_NCLK, ~KSP_COUNT_NCLK, ~KSP_INC_NCLK, ~SP_COUNT_NCLK, ~SP_INC_NCLK
- net labels removed: KSP_DEC_CLK, KSP_INC_CLK, PC_INC_CLK, SP_DEC_CLK, SP_INC_CLK
Other:
- note removed: "TODO: why is PC_INC, etc clocked?"
Changed lines of the file:
@@
 $Descr A3 16535 11693
 encoding utf-8
-Sheet 1 40
+Sheet 1 37
 Title ""
 Date ""
@@
 CLK
 $Sheet
-S 12750 5600 950  950
+S 12750 5600 950  1000
 U 5B0B7FE8
 F0 "Kernel Stack Register" 50
@@
 F11 "BUS6" I R 13700 6300 50
 F12 "BUS7" I R 13700 6400 50
-F13 "DOWN_OR_UP" I L 12750 6100 50
-F14 "COUNT_CLK" I L 12750 6000 50
-F15 "~R0_OUT" I L 12750 5700 50
-F16 "~R1_OUT" I L 12750 5800 50
-F17 "~R2_OUT" I L 12750 5900 50
-$EndSheet
-$Sheet
-S 12800 4400 900  950
-U 5B0B7FFA
-F0 "User Stack Register" 50
-F1 "stack_register.sch" 50
-F2 "~R0_IN" I L 12800 5000 50
-F3 "~R2_IN" I L 12800 5200 50
-F4 "BUS0" I R 13700 4500 50
-F5 "BUS1" I R 13700 4600 50
-F6 "BUS2" I R 13700 4700 50
-F7 "BUS3" I R 13700 4800 50
-F8 "BUS4" I R 13700 4900 50
-F9 "BUS5" I R 13700 5000 50
-F10 "BUS6" I R 13700 5100 50
-F11 "BUS7" I R 13700 5200 50
-F12 "DOWN_OR_UP" I L 12800 4900 50
-F13 "COUNT_CLK" I L 12800 4800 50
-F14 "~R0_OUT" I L 12800 4500 50
-F15 "~R1_OUT" I L 12800 4600 50
-F16 "~R2_OUT" I L 12800 4700 50
-F17 "~R1_IN" I L 12800 5100 50
+F13 "~R0_OUT" I L 12750 5700 50
+F14 "~R1_OUT" I L 12750 5800 50
+F15 "~R2_OUT" I L 12750 5900 50
+F16 "CLK" I L 12750 6000 50
+F17 "~COUNT_ENABLE" I L 12750 6500 50
+F18 "~UP" I L 12750 6100 50
 $EndSheet
 Text Label 13700 5700 0    50   ~ 0
@@
 Text Label 3850 8050 0    50   ~ 0
 INT7_IN_CLK
-Text Label 3850 8150 0    50   ~ 0
-PC_INC_CLK
-Text Label 3850 8250 0    50   ~ 0
-SP_INC_CLK
-Text Label 3850 8350 0    50   ~ 0
-SP_DEC_CLK
-Text Label 3850 8450 0    50   ~ 0
-KSP_INC_CLK
-Text Label 3850 8550 0    50   ~ 0
-KSP_DEC_CLK
 Text Label 3850 8650 0    50   ~ 0
 ALU_FLAG_SET_CLK
@@
 Text Label 12550 3700 2    50   ~ 0
 ~UNSET_INT_ENABLE_SYNC
-Text Notes 14000 2850 0    50   ~ 0
+Text Notes 14000 2850 0    197  ~ 0
 TODO: output these onto the bus
 Text Label 13900 3050 0    50   ~ 0
@@
 Text Label 10100 1600 2    50   ~ 0
 DISP_IN_CLK
-Text Notes 4800 8000 0    50   ~ 0
-TODO: why is PC_INC, etc clocked?
 Text Label 1850 2650 2    50   ~ 0
 BUS0
@@
 F53 "INT6_IN_CLK" I R 3850 7950 50
 F54 "INT7_IN_CLK" I R 3850 8050 50
-F55 "PC_INC_CLK" I R 3850 8150 50
-F56 "SP_INC_CLK" I R 3850 8250 50
-F57 "SP_DEC_CLK" I R 3850 8350 50
-F58 "KSP_INC_CLK" I R 3850 8450 50
-F59 "KSP_DEC_CLK" I R 3850 8550 50
-F60 "ALU_FLAG_SET_CLK" I R 3850 8650 50
-F61 "INT0" I R 3850 8750 50
-F62 "INT0_LATCH" I L 1850 3850 50
-F63 "INT1_LATCH" I L 1850 3950 50
-F64 "INT2_LATCH" I L 1850 4050 50
-F65 "INT3_LATCH" I L 1850 4150 50
-F66 "INT4_LATCH" I L 1850 4250 50
-F67 "INT5_LATCH" I L 1850 4350 50
-F68 "INT6_LATCH" I L 1850 4450 50
-F69 "INT7_LATCH" I L 1850 4550 50
-F70 "INTERRUPT_ENABLE_FLAG" I L 1850 4650 50
-F71 "MLU_SEL0" I R 3850 8850 50
-F72 "MLU_SEL1" I R 3850 8950 50
-F73 "MLU_SEL2" I R 3850 9050 50
-F74 "~PC0_OUT_NCLK" I R 3850 3850 50
-F75 "~PC1_OUT_NCLK" I R 3850 3950 50
-F76 "~PC2_OUT_NCLK" I R 3850 4050 50
-F77 "CLK" I L 1850 3750 50
-F78 "SUB_NCLK" I R 3850 4750 50
-F79 "~S0_IN_CLK" I R 3850 5750 50
-F80 "~S1_IN_CLK" I R 3850 5850 50
-F81 "~S2_IN_CLK" I R 3850 5950 50
-F82 "~K0_IN_CLK" I R 3850 6050 50
-F83 "~K1_IN_CLK" I R 3850 6150 50
-F84 "~K2_IN_CLK" I R 3850 6250 50
-F85 "~PC0_IN_NCLK" I R 3850 6350 50
-F86 "~PC1_IN_NCLK" I R 3850 6450 50
-F87 "~PC2_IN_NCLK" I R 3850 6550 50
+F55 "ALU_FLAG_SET_CLK" I R 3850 8650 50
+F56 "INT0" I R 3850 8750 50
+F57 "INT0_LATCH" I L 1850 3850 50
+F58 "INT1_LATCH" I L 1850 3950 50
+F59 "INT2_LATCH" I L 1850 4050 50
+F60 "INT3_LATCH" I L 1850 4150 50
+F61 "INT4_LATCH" I L 1850 4250 50
+F62 "INT5_LATCH" I L 1850 4350 50
+F63 "INT6_LATCH" I L 1850 4450 50
+F64 "INT7_LATCH" I L 1850 4550 50
+F65 "INTERRUPT_ENABLE_FLAG" I L 1850 4650 50
+F66 "MLU_SEL0" I R 3850 8850 50
+F67 "MLU_SEL1" I R 3850 8950 50
+F68 "MLU_SEL2" I R 3850 9050 50
+F69 "~PC0_OUT_NCLK" I R 3850 3850 50
+F70 "~PC1_OUT_NCLK" I R 3850 3950 50
+F71 "~PC2_OUT_NCLK" I R 3850 4050 50
+F72 "CLK" I L 1850 3750 50
+F73 "SUB_NCLK" I R 3850 4750 50
+F74 "~S0_IN_CLK" I R 3850 5750 50
+F75 "~S1_IN_CLK" I R 3850 5850 50
+F76 "~S2_IN_CLK" I R 3850 5950 50
+F77 "~K0_IN_CLK" I R 3850 6050 50
+F78 "~K1_IN_CLK" I R 3850 6150 50
+F79 "~K2_IN_CLK" I R 3850 6250 50
+F80 "~PC0_IN_NCLK" I R 3850 6350 50
+F81 "~PC1_IN_NCLK" I R 3850 6450 50
+F82 "~PC2_IN_NCLK" I R 3850 6550 50
+F83 "PC_INC_NCLK" I R 3850 8150 50
+F84 "~SP_COUNT_NCLK" I R 3850 8250 50
+F85 "~KSP_COUNT_NCLK" I R 3850 8450 50
+F86 "~SP_INC_NCLK" I R 3850 8350 50
+F87 "~KSP_INC_NCLK" I R 3850 8550 50
 $EndSheet
 Text Label 3850 6350 0    50   ~ 0
@@
 Text Label 12750 6400 2    50   ~ 0
 ~K2_IN_CLK
+Text Label 3850 8150 0    50   ~ 0
+PC_INC_NCLK
+Text Label 6400 5950 2    50   ~ 0
+PC_INC_NCLK
+$Sheet
+S 12800 4400 950  1000
+U 5B0B7FFA
+F0 "User Stack Register" 50
+F1 "stack_register.sch" 50
+F2 "~R0_IN" I L 12800 5000 50
+F3 "~R2_IN" I L 12800 5200 50
+F4 "BUS0" I R 13750 4500 50
+F5 "BUS1" I R 13750 4600 50
+F6 "BUS2" I R 13750 4700 50
+F7 "BUS3" I R 13750 4800 50
+F8 "BUS4" I R 13750 4900 50
+F9 "BUS5" I R 13750 5000 50
+F10 "BUS6" I R 13750 5100 50
+F11 "BUS7" I R 13750 5200 50
+F12 "~R0_OUT" I L 12800 4500 50
+F13 "~R1_OUT" I L 12800 4600 50
+F14 "~R2_OUT" I L 12800 4700 50
+F15 "~R1_IN" I L 12800 5100 50
+F16 "CLK" I L 12800 4800 50
+F17 "~COUNT_ENABLE" I L 12800 5300 50
+F18 "~UP" I L 12800 4900 50
+$EndSheet
+Text Label 12800 4800 2    50   ~ 0
+CLK
+Text Label 12750 6000 2    50   ~ 0
+CLK
+Text Label 3850 8250 0    50   ~ 0
+~SP_COUNT_NCLK
+Text Label 3850 8350 0    50   ~ 0
+~SP_INC_NCLK
+Text Label 3850 8450 0    50   ~ 0
+~KSP_COUNT_NCLK
+Text Label 3850 8550 0    50   ~ 0
+~KSP_INC_NCLK
+Text Label 12800 5300 2    50   ~ 0
+~SP_COUNT_NCLK
+Text Label 12800 4900 2    50   ~ 0
+~SP_INC_NCLK
+Text Label 12750 6500 2    50   ~ 0
+~KSP_COUNT_NCLK
+Text Label 12750 6100 2    50   ~ 0
+~KSP_INC_NCLK
 $EndSCHEMATC
