File: kicad/program_counter.sch (KiCad schematic (older format))
At the start: 18 parts

Commit message: Add SC register and program counter.
Parts:
- C47, C48, C49, C50, C51, C52: renamed from C?; value C_Small -> 0.1uF; footprint (none) -> Capacitor_THT:C_Disc_D3.0mm_W2.0mm_P2.50mm
- U39, U40, U41, U42, U43, U44: renamed from U?; footprint (none) -> Package_DIP:DIP-16_W7.62mm_Socket
- gave numbers to parts that had none: 6
Connections:
- net labels added: CARRY0, CARRY1, CARRY2, CARRY3, CARRY4, CLK, PC0_OUT, PC1_OUT, PC2_OUT, PC_INC
- net labels removed: REG_OUT
- wire segments 21 -> 18
Other:
- note removed: "TODO: there's an AND gate. Confirm with computer circuit."

Commit message: Schematic for kernel and user stack pointers.
Connections:
- net labels added: ~PC0_IN, ~PC0_OUT, ~PC1_IN, ~PC1_OUT, ~PC2_IN, ~PC2_OUT
- net labels removed: PC0_IN, PC0_OUT, PC1_IN, PC1_OUT, PC2_IN, PC2_OUT
Changed lines of the file:
@@
 $Descr A4 11693 8268
 encoding utf-8
-Sheet 17 17
+Sheet 17 19
 Title ""
 Date ""
@@
 Connection ~ 3900 3600
 Text HLabel 5650 2350 0    50   Input ~ 0
-PC0_OUT
+~PC0_OUT
 $Comp
 L 74xx:74HC245 U?
@@
 $EndComp
 Text HLabel 7800 2350 0    50   Input ~ 0
-PC1_OUT
+~PC1_OUT
 $Comp
 L 74xx:74HC245 U?
@@
 $EndComp
 Text HLabel 9850 2350 0    50   Input ~ 0
-PC2_OUT
+~PC2_OUT
 $Comp
 L 74xx:74HC245 U?
@@
 PC23
 Text HLabel 1550 1900 0    50   Input ~ 0
-PC0_IN
+~PC0_IN
 Text HLabel 3400 1900 0    50   Input ~ 0
-PC0_IN
+~PC0_IN
 Text HLabel 1550 4400 0    50   Input ~ 0
-PC1_IN
+~PC1_IN
 Text HLabel 3400 4400 0    50   Input ~ 0
-PC1_IN
+~PC1_IN
 Text HLabel 1500 6700 0    50   Input ~ 0
-PC2_IN
+~PC2_IN
 Text HLabel 3450 6700 0    50   Input ~ 0
-PC2_IN
+~PC2_IN
 Text Label 2550 1400 0    50   ~ 0
 PC0
@@
 Text Label 2550 1700 0    50   ~ 0
 PC3
-Text Label 4400 1450 0    50   ~ 0
+Text Label 4400 1400 0    50   ~ 0
 PC4
-Text Label 4400 1550 0    50   ~ 0
+Text Label 4400 1500 0    50   ~ 0
 PC5
-Text Label 4400 1650 0    50   ~ 0
+Text Label 4400 1600 0    50   ~ 0
 PC6
-Text Label 4400 1750 0    50   ~ 0
+Text Label 4400 1700 0    50   ~ 0
 PC7
 Text Label 2550 3900 0    50   ~ 0

Commit message: Control logic progress.
Connections:
- net labels added: ~PC0_IN_NCLK, ~PC1_IN_NCLK, ~PC2_IN_NCLK
- net labels removed: ~PC0_IN, ~PC1_IN, ~PC2_IN
Changed lines of the file:
@@
 PC23
 Text HLabel 1550 1900 0    50   Input ~ 0
-~PC0_IN
+~PC0_IN_NCLK
 Text HLabel 3400 1900 0    50   Input ~ 0
-~PC0_IN
+~PC0_IN_NCLK
 Text HLabel 1550 4400 0    50   Input ~ 0
-~PC1_IN
+~PC1_IN_NCLK
 Text HLabel 3400 4400 0    50   Input ~ 0
-~PC1_IN
+~PC1_IN_NCLK
 Text HLabel 1500 6700 0    50   Input ~ 0
-~PC2_IN
+~PC2_IN_NCLK
 Text HLabel 3450 6700 0    50   Input ~ 0
-~PC2_IN
+~PC2_IN_NCLK
 Text Label 2550 1400 0    50   ~ 0
 PC0
