File: kicad/_autosave-cpu.kicad_pcb (KiCad board)
At the start: 2 copper layers, 406 parts, among them J1 Conn_01x05, SW1 SW_DIP_x03 - Clock Source Sel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, SW2 SW_Push, SW3 SW_DPST, SW4 SW_Push, SW5 SW_DIP_x03, U1 LM555 - Adjustable Clock, U10 74HCT574, U100 74LS08, U101 74LS08, U102 74LS08, U105 74LS161, U106 74LS161, U107 74LS161, U108 74HC04, U109 74HC04, U11 74HC245, U110 74HC04, U111 74HC04, U112 74LS574, U113 SST39SF040, U114 74HC04, U115 74HC04, U117 74LS08, U118 74HC245, U119 74LS32, U12 74HCT574, U120 74LS32, U121 74HCT574, U122 74HC245, U123 74LS08, U125 74HC04, U13 74HC86, U14 74HCT574, U15 74HC86, U16 74HCT574, U17 74LS283, U18 74HCT574, U19 74LS283, U2 74HC14, U20 74HC245, U21 LM555, U22 74LS107, U23 74LS139, U24 AT28C64B, U25 HDSP-7803, U26 HDSP-7803, U27 HDSP-7803, U28 HDSP-7803, U29 74HCT574, U3 74151, U30 74HC86, U31 SST39SF040, U32 74LS107, U33 74LS08, U34 74LS107, U35 74LS107, U36 74HC00, U37 74HC74, U38 74HC74, U39 74LS161, U4 LM555 - Button Clock, U40 74LS161, U41 74LS161, U42 74LS161, U43 74LS161, U44 74LS161, U45 74HC245, U46 74HC245, U47 74HC245, U48 74LS191, U49 74LS191, U5 74HC04, U50 74LS191, U51 74LS191, U52 74LS191, U53 74LS191, U54 74LS08, U55 74HC04, U56 74HC245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

Commit message: Fix LEDs a bit.
Parts:
- moved D100 441.3 mm to (70.0, 306.0)
- moved D101 441.3 mm to (75.0, 306.0)
- moved D102 441.3 mm to (80.0, 306.0)
- moved D103 441.3 mm to (85.0, 306.0)
- moved D104 441.3 mm to (90.0, 306.0)
- moved D105 441.3 mm to (95.0, 306.0)
- moved D18 441.3 mm to (15.0, 276.0)
- moved D19 441.3 mm to (20.0, 276.0)
- moved D20 441.3 mm to (25.0, 276.0)
- moved D21 441.3 mm to (30.0, 276.0)
- moved D22 441.3 mm to (35.0, 276.0)
- moved D23 441.3 mm to (40.0, 276.0)
- moved D24 441.3 mm to (45.0, 276.0)
- moved D25 441.3 mm to (50.0, 276.0)
- moved D26 441.3 mm to (55.0, 276.0)
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Other:
- board text added: "Display module"
- board text added: "Power Circuitry"
- board text removed: "Manual Bus Input"
