File: kicad/control_logic.sch (KiCad schematic (older format))
At the start: 32 parts, among them U108 74HC04, U109 74HC04, U110 74HC04, U111 74HC04, U112 74LS574, U113 SST39SF040, U114 74HC04, U115 74HC04, U117 74LS08, U118 74HC245, U125 74HC04, U5 74HC04, U87 74LS574, U88 SST39SF040, U89 74LS574, U90 SST39SF040, U92 74LS154

Commit message: Reset related progress.
Parts:
- removed unit 4 of U117
Connections:
- net labels added: ~RESET
- no-connect marks 7 -> 6
Other:
- note added: "TODO: Move spares from other locations back?"
- note added: "Update the micro-op counter on the rising edge so\nwe have enough time to latch the control word on\nthe falling edge (not trying to simultaneously \nupdate the micro op counter)."
- note removed: "TODO: CLK or ~CLK?"
- note removed: "TODO: Move spares back?"
- moved on the sheet: U125A, U125B, U125C, U125D, U125E, U125F
Changed lines of the file:
@@
 $Descr A3 16535 11693
 encoding utf-8
-Sheet 24 36
+Sheet 23 36
 Title ""
 Date ""
@@
 Text HLabel 8450 4850 2    50   Input ~ 0
 ~RESET_NCLK
-Text HLabel 8450 4950 2    50   Input ~ 0
-~RESET_UOP_COUNT_NCLK
 Text HLabel 8450 5050 2    50   Input ~ 0
 ~SET_INT_ENABLE_SYNC
@@
 F1 "microop_counter.sch" 50
 F2 "~RESET" I L 12500 1450 50
-F3 "~CLK" I L 12500 1550 50
+F3 "CLK" I L 12500 1550 50
 F4 "O0" I R 13050 1450 50
 F5 "O1" I R 13050 1550 50
@@
 $Comp
 L 74xx:74LS08 U117
-U 4 1 5B1CDA04
-P 18500 9600
-F 0 "U117" H 18500 9925 50  0000 C CNN
-F 1 "74LS08" H 18500 9834 50  0000 C CNN
-F 2 "" H 18500 9600 50  0001 C CNN
-F 3 "http://www.ti.com/lit/gpn/sn74LS08" H 18500 9600 50  0001 C CNN
-	4    18500 9600
-	1    0    0    -1
-$EndComp
-$Comp
-L 74xx:74LS08 U117
 U 5 1 5B1CDB22
 P 9250 -50
@@
 Text Notes 18400 8400 0    50   ~ 0
 Spares
-$Comp
-L power:GND #PWR0457
-U 1 1 5B1D9C5A
-P 17100 9000
-F 0 "#PWR0457" H 17100 8750 50  0001 C CNN
-F 1 "GND" V 17105 8872 50  0000 R CNN
-F 2 "" H 17100 9000 50  0001 C CNN
-F 3 "" H 17100 9000 50  0001 C CNN
-	1    17100 9000
-	0    1    1    0
-$EndComp
-$Comp
-L power:GND #PWR0458
-U 1 1 5B1D9D03
-P 17100 9200
-F 0 "#PWR0458" H 17100 8950 50  0001 C CNN
-F 1 "GND" V 17105 9072 50  0000 R CNN
-F 2 "" H 17100 9200 50  0001 C CNN
-F 3 "" H 17100 9200 50  0001 C CNN
-	1    17100 9200
-	0    1    1    0
-$EndComp
-$Comp
-L power:GND #PWR0459
-U 1 1 5B1D9DAC
-P 17100 9500
-F 0 "#PWR0459" H 17100 9250 50  0001 C CNN
-F 1 "GND" V 17105 9372 50  0000 R CNN
-F 2 "" H 17100 9500 50  0001 C CNN
-F 3 "" H 17100 9500 50  0001 C CNN
-	1    17100 9500
-	0    1    1    0
-$EndComp
-$Comp
-L power:GND #PWR0460
-U 1 1 5B1D9E55
-P 17100 9700
-F 0 "#PWR0460" H 17100 9450 50  0001 C CNN
-F 1 "GND" V 17105 9572 50  0000 R CNN
-F 2 "" H 17100 9700 50  0001 C CNN
-F 3 "" H 17100 9700 50  0001 C CNN
-	1    17100 9700
-	0    1    1    0
-$EndComp
-$Comp
-L power:GND #PWR0461
-U 1 1 5B1D9EFE
-P 18200 9500
-F 0 "#PWR0461" H 18200 9250 50  0001 C CNN
-F 1 "GND" V 18205 9372 50  0000 R CNN
-F 2 "" H 18200 9500 50  0001 C CNN
-F 3 "" H 18200 9500 50  0001 C CNN
-	1    18200 9500
-	0    1    1    0
-$EndComp
-$Comp
-L power:GND #PWR0462
-U 1 1 5B1D9FA7
-P 18200 9700
-F 0 "#PWR0462" H 18200 9450 50  0001 C CNN
-F 1 "GND" V 18205 9572 50  0000 R CNN
-F 2 "" H 18200 9700 50  0001 C CNN
-F 3 "" H 18200 9700 50  0001 C CNN
-	1    18200 9700
-	0    1    1    0
-$EndComp
-NoConn ~ 18800 9600
 Text HLabel 4200 2500 2    50   Input ~ 0
 MLU_SEL0
@@
 L 74xx:74HC04 U125
 U 1 1 5B250A2C
-P 15850 7850
-F 0 "U125" H 15850 7850 50  0000 C CNN
-F 1 "74HC04" H 16000 7750 50  0000 C CNN
-F 2 "" H 15850 7850 50  0001 C CNN
-F 3 "http://www.nxp.com/documents/data_sheet/74HC_HCT04.pdf" H 15850 7850 50  0001 C CNN
-	1    15850 7850
+P 14100 7850
+F 0 "U125" H 14100 7850 50  0000 C CNN
+F 1 "74HC04" H 14250 7750 50  0000 C CNN
+F 2 "" H 14100 7850 50  0001 C CNN
+F 3 "http://www.nxp.com/documents/data_sheet/74HC_HCT04.pdf" H 14100 7850 50  0001 C CNN
+	1    14100 7850
 	1    0    0    -1
 $EndComp
@@
 L 74xx:74HC04 U125
 U 2 1 5B250A33
-P 15850 8150
-F 0 "U125" H 15850 8150 50  0000 C CNN
-F 1 "74HC04" H 16000 8050 50  0000 C CNN
-F 2 "" H 15850 8150 50  0001 C CNN
-F 3 "http://www.nxp.com/documents/data_sheet/74HC_HCT04.pdf" H 15850 8150 50  0001 C CNN
-	2    15850 8150
+P 14100 8150
+F 0 "U125" H 14100 8150 50  0000 C CNN
+F 1 "74HC04" H 14250 8050 50  0000 C CNN
+F 2 "" H 14100 8150 50  0001 C CNN
+F 3 "http://www.nxp.com/documents/data_sheet/74HC_HCT04.pdf" H 14100 8150 50  0001 C CNN
+	2    14100 8150
 	1    0    0    -1
 $EndComp
@@
 L 74xx:74HC04 U125
 U 3 1 5B250A3A
-P 15850 8450
-F 0 "U125" H 15850 8450 50  0000 C CNN
-F 1 "74HC04" H 16000 8350 50  0000 C CNN
-F 2 "" H 15850 8450 50  0001 C CNN
-F 3 "http://www.nxp.com/documents/data_sheet/74HC_HCT04.pdf" H 15850 8450 50  0001 C CNN
-	3    15850 8450
+P 14100 8450
+F 0 "U125" H 14100 8450 50  0000 C CNN
+F 1 "74HC04" H 14250 8350 50  0000 C CNN
+F 2 "" H 14100 8450 50  0001 C CNN
+F 3 "http://www.nxp.com/documents/data_sheet/74HC_HCT04.pdf" H 14100 8450 50  0001 C CNN
+	3    14100 8450
 	1    0    0    -1
 $EndComp
@@
 L 74xx:74HC04 U125
 U 4 1 5B250A41
-P 15850 8750
-F 0 "U125" H 15850 8750 50  0000 C CNN
-F 1 "74HC04" H 16000 8650 50  0000 C CNN
-F 2 "" H 15850 8750 50  0001 C CNN
-F 3 "http://www.nxp.com/documents/data_sheet/74HC_HCT04.pdf" H 15850 8750 50  0001 C CNN
-	4    15850 8750
+P 14100 8750
+F 0 "U125" H 14100 8750 50  0000 C CNN
+F 1 "74HC04" H 14250 8650 50  0000 C CNN
+F 2 "" H 14100 8750 50  0001 C CNN
+F 3 "http://www.nxp.com/documents/data_sheet/74HC_HCT04.pdf" H 14100 8750 50  0001 C CNN
+	4    14100 8750
 	1    0    0    -1
 $EndComp
@@
 L 74xx:74HC04 U125
 U 5 1 5B250A48
-P 15850 9050
-F 0 "U125" H 15850 9050 50  0000 C CNN
-F 1 "74HC04" H 16000 8950 50  0000 C CNN
-F 2 "" H 15850 9050 50  0001 C CNN
-F 3 "http://www.nxp.com/documents/data_sheet/74HC_HCT04.pdf" H 15850 9050 50  0001 C CNN
-	5    15850 9050
+P 14100 9050
+F 0 "U125" H 14100 9050 50  0000 C CNN
+F 1 "74HC04" H 14250 8950 50  0000 C CNN
+F 2 "" H 14100 9050 50  0001 C CNN
+F 3 "http://www.nxp.com/documents/data_sheet/74HC_HCT04.pdf" H 14100 9050 50  0001 C CNN
+	5    14100 9050
 	1    0    0    -1
 $EndComp
@@
 L 74xx:74HC04 U125
 U 6 1 5B250A4F
-P 15850 9350
-F 0 "U125" H 15850 9350 50  0000 C CNN
-F 1 "74HC04" H 16000 9250 50  0000 C CNN
-F 2 "" H 15850 9350 50  0001 C CNN
-F 3 "http://www.nxp.com/documents/data_sheet/74HC_HCT04.pdf" H 15850 9350 50  0001 C CNN
-	6    15850 9350
+P 14100 9350
+F 0 "U125" H 14100 9350 50  0000 C CNN
+F 1 "74HC04" H 14250 9250 50  0000 C CNN
+F 2 "" H 14100 9350 50  0001 C CNN
+F 3 "http://www.nxp.com/documents/data_sheet/74HC_HCT04.pdf" H 14100 9350 50  0001 C CNN
+	6    14100 9350
 	1    0    0    -1
 $EndComp
@@
 Text Label 6400 10050 0    50   ~ 0
 K2_IN_CLK
-Text Label 15550 7850 2    50   ~ 0
+Text Label 13800 7850 2    50   ~ 0
 S0_IN_CLK
-Text Label 15550 8150 2    50   ~ 0
+Text Label 13800 8150 2    50   ~ 0
 S1_IN_CLK
-Text Label 15550 8450 2    50   ~ 0
+Text Label 13800 8450 2    50   ~ 0
 S2_IN_CLK
 Text Notes 14400 4400 0    50   ~ 0
 SUB is active high.
-Text Notes 15100 7550 0    50   ~ 0
+Text Notes 13350 7550 0    50   ~ 0
 Stack registers are presettable.\nBut, they read asynchronously\non an active low signal. So, invert.
-Text Label 15550 8750 2    50   ~ 0
+Text Label 13800 8750 2    50   ~ 0
 K0_IN_CLK
-Text Label 15550 9050 2    50   ~ 0
+Text Label 13800 9050 2    50   ~ 0
 K1_IN_CLK
-Text Label 15550 9350 2    50   ~ 0
+Text Label 13800 9350 2    50   ~ 0
 K2_IN_CLK
-Text HLabel 16150 7850 2    50   Input ~ 0
+Text HLabel 14400 7850 2    50   Input ~ 0
 ~S0_IN_CLK
-Text HLabel 16150 8150 2    50   Input ~ 0
+Text HLabel 14400 8150 2    50   Input ~ 0
 ~S1_IN_CLK
-Text HLabel 16150 8450 2    50   Input ~ 0
+Text HLabel 14400 8450 2    50   Input ~ 0
 ~S2_IN_CLK
-Text HLabel 16150 8750 2    50   Input ~ 0
+Text HLabel 14400 8750 2    50   Input ~ 0
 ~K0_IN_CLK
-Text HLabel 16150 9050 2    50   Input ~ 0
+Text HLabel 14400 9050 2    50   Input ~ 0
 ~K1_IN_CLK
-Text HLabel 16150 9350 2    50   Input ~ 0
+Text HLabel 14400 9350 2    50   Input ~ 0
 ~K2_IN_CLK
 Text HLabel 2350 9050 2    50   Input ~ 0
@@
 Text HLabel 6400 10850 2    50   Input ~ 0
 MMU_CONTROL_IN_CLK
-Text Notes 11800 9800 0    157  ~ 0
-TODO: Move spares back?
+Text Notes 16650 8000 0    157  ~ 0
+TODO: Move spares from other locations back?
 Text Label 10400 2550 2    50   ~ 0
 OPCODE0_INC_NCLK
 Text Label 10400 2750 2    50   ~ 0
 OPCODE1_INC_NCLK
-Text Notes 9550 1250 0    157  ~ 0
-TODO: CLK or ~CLK?
 Text HLabel 10950 4700 2    50   Input ~ 0
 PC_INC_NCLK
@@
 Text HLabel 8450 5750 2    50   Input ~ 0
 ~KSP_INC_NCLK
+Text HLabel 10400 2350 0    50   Input ~ 0
+~RESET
+Text HLabel 10400 2450 0    50   Input ~ 0
+CLK
+Text Label 8450 4950 0    50   ~ 0
+~RESET_UOP_COUNT_NCLK
+Text Label 12500 1450 2    50   ~ 0
+~RESET_UOP_COUNT_NCLK
+Text Notes 11950 1200 0    50   ~ 0
+Update the micro-op counter on the rising edge so\nwe have enough time to latch the control word on\nthe falling edge (not trying to simultaneously \nupdate the micro op counter).
+Text Label 12500 1550 2    50   ~ 0
+CLK
 $EndSCHEMATC

Commit message: Small update.
Connections:
- no-connect marks 6 -> 9
Changed lines of the file:
@@
 Text Label 12500 1550 2    50   ~ 0
 CLK
+$Comp
+L power:GND #PWR0454
+U 1 1 5B40242D
+P 17300 8450
+F 0 "#PWR0454" H 17300 8200 50  0001 C CNN
+F 1 "GND" V 17305 8322 50  0000 R CNN
+F 2 "" H 17300 8450 50  0001 C CNN
+F 3 "" H 17300 8450 50  0001 C CNN
+	1    17300 8450
+	0    1    1    0
+$EndComp
+NoConn ~ 17900 8450
+$Comp
+L power:GND #PWR0457
+U 1 1 5B40299A
+P 18150 8600
+F 0 "#PWR0457" H 18150 8350 50  0001 C CNN
+F 1 "GND" V 18155 8472 50  0000 R CNN
+F 2 "" H 18150 8600 50  0001 C CNN
+F 3 "" H 18150 8600 50  0001 C CNN
+	1    18150 8600
+	0    1    1    0
+$EndComp
+$Comp
+L power:GND #PWR0458
+U 1 1 5B402A3D
+P 18150 8900
+F 0 "#PWR0458" H 18150 8650 50  0001 C CNN
+F 1 "GND" V 18155 8772 50  0000 R CNN
+F 2 "" H 18150 8900 50  0001 C CNN
+F 3 "" H 18150 8900 50  0001 C CNN
+	1    18150 8900
+	0    1    1    0
+$EndComp
+NoConn ~ 18750 8600
+NoConn ~ 18750 8900
 $EndSCHEMATC

Commit message: Import into pcbnew.
Parts:
- U108, U109, U110, U111, U114, U115, U117, U125: footprint (none) -> Package_DIP:DIP-14_W7.62mm_Socket
- U118: footprint (none) -> Package_DIP:DIP-20_W7.62mm_Socket
Other:
- note removed: "TODO: INT0_IN_CLK should be unconnected - should get a warning about it."

Commit message: Layout progress.
Parts:
- added C127: 0.1uF, Capacitor_THT:C_Disc_D3.0mm_W2.0mm_P2.50mm, symbol Device:C_Small
- added unit 7 of U125
Connections:
- wire segments 23 -> 24
Changed lines of the file:
@@
 NoConn ~ 18750 8600
 NoConn ~ 18750 8900
+$Comp
+L 74xx:74HC04 U125
+U 7 1 5B15AA5E
+P 8100 -100
+F 0 "U125" H 8330 -54 50  0000 L CNN
+F 1 "74HC04" H 8330 -145 50  0000 L CNN
+F 2 "Package_DIP:DIP-14_W7.62mm_Socket" H 8100 -100 50  0001 C CNN
+F 3 "http://www.nxp.com/documents/data_sheet/74HC_HCT04.pdf" H 8100 -100 50  0001 C CNN
+	7    8100 -100
+	1    0    0    -1
+$EndComp
+$Comp
+L power:VCC #PWR058
+U 1 1 5B15AA65
+P 8100 -600
+F 0 "#PWR058" H 8100 -750 50  0001 C CNN
+F 1 "VCC" H 8117 -427 50  0000 C CNN
+F 2 "" H 8100 -600 50  0001 C CNN
+F 3 "" H 8100 -600 50  0001 C CNN
+	1    8100 -600
+	1    0    0    -1
+$EndComp
+$Comp
+L Device:C_Small C127
+U 1 1 5B15AA6B
+P 8450 -600
+F 0 "C127" V 8221 -600 50  0000 C CNN
+F 1 "0.1uF" V 8312 -600 50  0000 C CNN
+F 2 "Capacitor_THT:C_Disc_D3.0mm_W2.0mm_P2.50mm" H 8450 -600 50  0001 C CNN
+F 3 "~" H 8450 -600 50  0001 C CNN
+	1    8450 -600
+	0    1    1    0
+$EndComp
+$Comp
+L power:GND #PWR060
+U 1 1 5B15AA72
+P 8550 -600
+F 0 "#PWR060" H 8550 -850 50  0001 C CNN
+F 1 "GND" V 8555 -728 50  0000 R CNN
+F 2 "" H 8550 -600 50  0001 C CNN
+F 3 "" H 8550 -600 50  0001 C CNN
+	1    8550 -600
+	0    -1   -1   0
+$EndComp
+Wire Wire Line
+	8100 -600 8350 -600
+Connection ~ 8100 -600
+$Comp
+L power:GND #PWR059
+U 1 1 5B15AA7A
+P 8100 400
+F 0 "#PWR059" H 8100 150 50  0001 C CNN
+F 1 "GND" V 8105 272 50  0000 R CNN
+F 2 "" H 8100 400 50  0001 C CNN
+F 3 "" H 8100 400 50  0001 C CNN
+	1    8100 400
+	1    0    0    -1
+$EndComp
 $EndSCHEMATC

Commit message: Add control logic LEDs to schematic.
Parts:
- removed U5: 74HC04, Package_DIP:DIP-14_W7.62mm_Socket, symbol 74xx:74HC04
Connections:
- net labels added: ~SET_INT_ENABLE_ASYNC, ~UNSET_INT_ENABLE_ASYNC
- net labels removed: INT0, ~SET_INT_ENABLE_SYNC, ~UNSET_INT_ENABLE_SYNC
Other:
- note added: "TODO: Connect these and INs, \nand interrupt lines up to\nboard interconnect.\n"
- note removed: "Software interrupt line - INT0"
- note removed: "TODO: Move spares from other locations back?"
- note removed: "Taken from spares \nfrom clock"
- moved on the sheet: U108A, U108B, U108C, U108D, U108E, U108F, U108G, U109A, U109B, U109C, U109D, U109E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

Commit message: Going to try out resistor network.
Connections:
- net labels added: OPCODE0_IN_NCLK, OPCODE1_IN_NCLK, PC0_IN_NCLK, PC1_IN_NCLK, PC2_IN_NCLK
Changed lines of the file:
@@
 $EndComp
 $Sheet
-S 18450 4150 1550 5300
+S 18450 4150 1900 4600
 U 5B1644E8
 F0 "Control Logic LEDs" 50
@@
 F31 "INT6_IN" I L 18450 7150 50
 F32 "INT7_IN" I L 18450 7250 50
+F33 "~A_OUT" I R 20350 4250 50
+F34 "~B_OUT" I R 20350 4350 50
+F35 "~M0_OUT" I R 20350 4450 50
+F36 "~M1_OUT" I R 20350 4550 50
+F37 "~M2_OUT" I R 20350 4650 50
+F38 "~S0_OUT" I R 20350 4750 50
+F39 "~S1_OUT" I R 20350 4850 50
+F40 "~S2_OUT" I R 20350 4950 50
+F41 "~K0_OUT" I R 20350 5050 50
+F42 "~K1_OUT" I R 20350 5150 50
+F43 "~K2_OUT" I R 20350 5250 50
+F44 "~PC0_OUT" I R 20350 5350 50
+F45 "~PC1_OUT" I R 20350 5450 50
+F46 "~PC2_OUT" I R 20350 5550 50
+F47 "~STATUS_OUT" I R 20350 5650 50
+F48 "~INTERRUPT_OUT" I R 20350 5750 50
+F49 "~SUM_OUT" I R 20350 5850 50
+F50 "~MMU_OUT" I R 20350 5950 50
+F51 "~MMU_CONTROL_OUT" I R 20350 6050 50
+F52 "~TASK_OUT" I R 20350 6150 50
+F53 "~MLU_OUT" I R 20350 6250 50
+F54 "~CTRLLOGIC_OUT" I R 20350 6350 50
+F55 "~INT1_OUT" I R 20350 6550 50
+F56 "~INT2_OUT" I R 20350 6650 50
+F57 "~INT3_OUT" I R 20350 6750 50
+F58 "~INT4_OUT" I R 20350 6850 50
+F59 "~INT5_OUT" I R 20350 6950 50
+F60 "~INT6_OUT" I R 20350 7050 50
+F61 "~INT7_OUT" I R 20350 7150 50
+F62 "~INT0_OUT" I R 20350 6450 50
+F63 "SUB" I L 18450 7400 50
+F64 "~RESET" I L 18450 7500 50
+F65 "~RESET_UOP_COUNT" I L 18450 7600 50
+F66 "~SET_INT_ENABLE_ASYNC" I L 18450 7700 50
+F67 "~UNSET_INT_ENABLE_ASYNC" I L 18450 7800 50
+F68 "PC_INC" I L 18450 7900 50
+F69 "OPCODE0_INC" I L 18450 8000 50
+F70 "OPCODE1_INC" I L 18450 8100 50
+F71 "~SP_INC" I L 18450 8200 50
+F72 "~SP_DEC" I L 18450 8300 50
+F73 "~KSP_INC" I L 18450 8400 50
+F74 "~KSP_DEC" I L 18450 8500 50
+F75 "ALU_FLAG_SET" I L 18450 8600 50
+F76 "MICROOP0" I R 20350 7300 50
+F77 "MICROOP1" I R 20350 7400 50
+F78 "MICROOP2" I R 20350 7500 50
+F79 "MICROOP3" I R 20350 7600 50
+F80 "MMU_READ_FAULT" I R 20350 7700 50
+F81 "MMU_WRITE_FAULT" I R 20350 7800 50
+F82 "INT0_LATCH" I R 20350 7900 50
+F83 "INT1_LATCH" I R 20350 8000 50
+F84 "INT2_LATCH" I R 20350 8100 50
+F85 "INT3_LATCH" I R 20350 8200 50
+F86 "INT4_LATCH" I R 20350 8300 50
+F87 "INT5_LATCH" I R 20350 8400 50
+F88 "INT6_LATCH" I R 20350 8500 50
+F89 "INT7_LATCH" I R 20350 8600 50
 $EndSheet
 Text Notes 7150 5550 0    79   ~ 0
 TODO: Connect these and INs, \nand interrupt lines up to\nboard interconnect.\n
+Text Label 18450 4250 2    50   ~ 0
+A_IN_NCLK
+Text Label 18450 4350 2    50   ~ 0
+B_IN_NCLK
+Text Label 18450 4450 2    50   ~ 0
+M0_IN_NCLK
+Text Label 18450 4550 2    50   ~ 0
+M1_IN_NCLK
+Text Label 18450 4650 2    50   ~ 0
+M2_IN_NCLK
+Text Label 18450 4750 2    50   ~ 0
+S0_IN_NCLK
+Text Label 18450 4850 2    50   ~ 0
+S1_IN_NCLK
+Text Label 18450 4950 2    50   ~ 0
+S2_IN_NCLK
+Text Label 18450 5050 2    50   ~ 0
+K0_IN_NCLK
+Text Label 18450 5150 2    50   ~ 0
+K1_IN_NCLK
+Text Label 18450 5250 2    50   ~ 0
+K2_IN_NCLK
+Text Label 18450 5350 2    50   ~ 0
+PC0_IN_NCLK
+Text Label 18450 5450 2    50   ~ 0
+PC1_IN_NCLK
+Text Label 18450 5550 2    50   ~ 0
+PC2_IN_NCLK
+Text Label 18450 5650 2    50   ~ 0
+MMU0_IN_NCLK
+Text Label 18450 5750 2    50   ~ 0
+MMU1_IN_NCLK
+Text Label 18450 5850 2    50   ~ 0
+MMU2_IN_NCLK
+Text Label 18450 5950 2    50   ~ 0
+MMU_IN_NCLK
+Text Label 18450 6050 2    50   ~ 0
+MMU_CONTROL_IN_NCLK
+Text Label 18450 6150 2    50   ~ 0
+DISP_IN_NCLK
+Text Label 18450 6250 2    50   ~ 0
+TASK_IN_NCLK
+Text Label 18450 6350 2    50   ~ 0
+OPCODE0_IN_NCLK
+Text Label 18450 6450 2    50   ~ 0
+OPCODE1_IN_NCLK
+Text Label 18450 6550 2    50   ~ 0
+INT0_IN_NCLK
+Text Label 18450 6650 2    50   ~ 0
+INT1_IN_NCLK
+Text Label 18450 6750 2    50   ~ 0
+INT2_IN_NCLK
+Text Label 18450 6850 2    50   ~ 0
+INT3_IN_NCLK
+Text Label 18450 6950 2    50   ~ 0
+INT4_IN_NCLK
+Text Label 18450 7050 2    50   ~ 0
+INT5_IN_NCLK
+Text Label 18450 7150 2    50   ~ 0
+INT6_IN_NCLK
+Text Label 18450 7250 2    50   ~ 0
+INT7_IN_NCLK
+Text Label 20350 4250 0    50   ~ 0
+~A_OUT_NCLK
+Text Label 20350 4350 0    50   ~ 0
+~B_OUT_NCLK
+Text Label 20350 4450 0    50   ~ 0
+~M0_OUT_NCLK
+Text Label 20350 4550 0    50   ~ 0
+~M1_OUT_NCLK
+Text Label 20350 4650 0    50   ~ 0
+~M2_OUT_NCLK
+Text Label 20350 4750 0    50   ~ 0
+~S0_OUT_NCLK
+Text Label 20350 4850 0    50   ~ 0
+~S1_OUT_NCLK
+Text Label 20350 4950 0    50   ~ 0
+~S2_OUT_NCLK
+Text Label 20350 5050 0    50   ~ 0
+~K0_OUT_NCLK
+Text Label 20350 5150 0    50   ~ 0
+~K1_OUT_NCLK
+Text Label 20350 5250 0    50   ~ 0
+~K2_OUT_NCLK
+Text Label 20350 5350 0    50   ~ 0
+~PC0_OUT_NCLK
+Text Label 20350 5450 0    50   ~ 0
+~PC1_OUT_NCLK
+Text Label 20350 5550 0    50   ~ 0
+~PC2_OUT_NCLK
+Text Label 20350 5650 0    50   ~ 0
+~STATUS_OUT_NCLK
+Text Label 20350 5750 0    50   ~ 0
+~INTERRUPT_OUT_NCLK
+Text Label 20350 5850 0    50   ~ 0
+~SUM_OUT_NCLK
+Text Label 20350 5950 0    50   ~ 0
+~MMU_OUT_NCLK
+Text Label 20350 6050 0    50   ~ 0
+~MMU_CONTROL_OUT_NCLK
+Text Label 20350 6150 0    50   ~ 0
+~TASK_OUT_NCLK
+Text Label 20350 6250 0    50   ~ 0
+~MLU_OUT_NCLK
+Text Label 20350 6350 0    50   ~ 0
+~CTRLLOGIC_OUT_NCLK
+Text Label 20350 6450 0    50   ~ 0
+~INT0_OUT_NCLK
+Text Label 20350 6550 0    50   ~ 0
+~INT1_OUT_NCLK
+Text Label 20350 6650 0    50   ~ 0
+~INT2_OUT_NCLK
+Text Label 20350 6750 0    50   ~ 0
+~INT3_OUT_NCLK
+Text Label 20350 6850 0    50   ~ 0
+~INT4_OUT_NCLK
+Text Label 20350 6950 0    50   ~ 0
+~INT5_OUT_NCLK
+Text Label 20350 7050 0    50   ~ 0
+~INT6_OUT_NCLK
+Text Label 20350 7150 0    50   ~ 0
+~INT7_OUT_NCLK
+Text Label 18450 7400 2    50   ~ 0
+SUB_NCLK
+Text Label 18450 7500 2    50   ~ 0
+~RESET_NCLK
+Text Label 18450 7600 2    50   ~ 0
+~RESET_UOP_COUNT_NCLK
+Text Label 18450 7700 2    50   ~ 0
+~SET_INT_ENABLE_ASYNC
+Text Label 18450 7800 2    50   ~ 0
+~UNSET_INT_ENABLE_ASYNC
+Text Label 18450 7900 2    50   ~ 0
+PC_INC_NCLK
+Text Label 18450 8000 2    50   ~ 0
+OPCODE0_INC_NCLK
+Text Label 18450 8100 2    50   ~ 0
+OPCODE1_INC_NCLK
+Text Label 18450 8200 2    50   ~ 0
+~SP_INC_NCLK
+Text Label 18450 8300 2    50   ~ 0
+~SP_DEC_NCLK
+Text Label 18450 8400 2    50   ~ 0
+~KSP_INC_NCLK
+Text Label 18450 8500 2    50   ~ 0
+~KSP_DEC_NCLK
+Text Label 18450 8600 2    50   ~ 0
+ALU_FLAG_SET_NCLK
+Text Label 20350 7300 0    50   ~ 0
+MICROOP0
+Text Label 20350 7400 0    50   ~ 0
+MICROOP1
+Text Label 20350 7500 0    50   ~ 0
+MICROOP2
+Text Label 20350 7600 0    50   ~ 0
+MICROOP3
+Text Label 20350 7700 0    50   ~ 0
+MMU_READ_FAULT
+Text Label 20350 7800 0    50   ~ 0
+MMU_WRITE_FAULT
+Text Label 20350 7900 0    50   ~ 0
+INT0_LATCH
+Text Label 20350 8000 0    50   ~ 0
+INT1_LATCH
+Text Label 20350 8100 0    50   ~ 0
+INT2_LATCH
+Text Label 20350 8200 0    50   ~ 0
+INT3_LATCH
+Text Label 20350 8300 0    50   ~ 0
+INT4_LATCH
+Text Label 20350 8400 0    50   ~ 0
+INT5_LATCH
+Text Label 20350 8500 0    50   ~ 0
+INT6_LATCH
+Text Label 20350 8600 0    50   ~ 0
+INT7_LATCH
 $EndSCHEMATC

Commit message: Fix LEDs a bit.
Connections:
- net labels removed: OPCODE0_IN_NCLK, OPCODE1_IN_NCLK, PC0_IN_NCLK, PC1_IN_NCLK, PC2_IN_NCLK
Changed lines of the file:
@@
 Text Label 2000 11450 2    50   ~ 0
 ~INT7_IN_NCLK
-Text Label 8200 4300 2    50   ~ 0
-~INT0_OUT_NCLK
-Text Label 8200 4400 2    50   ~ 0
-~INT1_OUT_NCLK
-Text Label 8200 4500 2    50   ~ 0
-~INT2_OUT_NCLK
-Text Label 8200 4600 2    50   ~ 0
-~INT3_OUT_NCLK
-Text Label 8200 4700 2    50   ~ 0
-~INT4_OUT_NCLK
-Text Label 8200 4800 2    50   ~ 0
-~INT5_OUT_NCLK
-Text Label 8200 4900 2    50   ~ 0
-~INT6_OUT_NCLK
-Text Label 8200 5000 2    50   ~ 0
-~INT7_OUT_NCLK
 NoConn ~ 8200 4200
 $Comp
@@
 F11 "K1_IN" I L 18450 5150 50
 F12 "K2_IN" I L 18450 5250 50
-F13 "PC0_IN" I L 18450 5350 50
-F14 "PC1_IN" I L 18450 5450 50
-F15 "PC2_IN" I L 18450 5550 50
+F13 "~PC0_IN" I L 18450 5350 50
+F14 "~PC1_IN" I L 18450 5450 50
+F15 "~PC2_IN" I L 18450 5550 50
 F16 "MMU0_IN" I L 18450 5650 50
 F17 "MMU1_IN" I L 18450 5750 50
@@
 F21 "DISP_IN" I L 18450 6150 50
 F22 "TASK_IN" I L 18450 6250 50
-F23 "OPCODE0_IN" I L 18450 6350 50
-F24 "OPCODE1_IN" I L 18450 6450 50
+F23 "~OPCODE0_IN" I L 18450 6350 50
+F24 "~OPCODE1_IN" I L 18450 6450 50
 F25 "INT0_IN" I L 18450 6550 50
 F26 "INT1_IN" I L 18450 6650 50
@@
 Text Label 18450 5250 2    50   ~ 0
 K2_IN_NCLK
-Text Label 18450 5350 2    50   ~ 0
-PC0_IN_NCLK
-Text Label 18450 5450 2    50   ~ 0
-PC1_IN_NCLK
-Text Label 18450 5550 2    50   ~ 0
-PC2_IN_NCLK
 Text Label 18450 5650 2    50   ~ 0
 MMU0_IN_NCLK
@@
 TASK_IN_NCLK
 Text Label 18450 6350 2    50   ~ 0
-OPCODE0_IN_NCLK
+~OPCODE0_IN_NCLK
 Text Label 18450 6450 2    50   ~ 0
-OPCODE1_IN_NCLK
+~OPCODE1_IN_NCLK
 Text Label 18450 6550 2    50   ~ 0
 INT0_IN_NCLK
@@
 Text Label 20350 6350 0    50   ~ 0
 ~CTRLLOGIC_OUT_NCLK
-Text Label 20350 6450 0    50   ~ 0
-~INT0_OUT_NCLK
-Text Label 20350 6550 0    50   ~ 0
-~INT1_OUT_NCLK
-Text Label 20350 6650 0    50   ~ 0
-~INT2_OUT_NCLK
-Text Label 20350 6750 0    50   ~ 0
-~INT3_OUT_NCLK
-Text Label 20350 6850 0    50   ~ 0
-~INT4_OUT_NCLK
-Text Label 20350 6950 0    50   ~ 0
-~INT5_OUT_NCLK
-Text Label 20350 7050 0    50   ~ 0
-~INT6_OUT_NCLK
-Text Label 20350 7150 0    50   ~ 0
-~INT7_OUT_NCLK
 Text Label 18450 7400 2    50   ~ 0
 SUB_NCLK
@@
 Text Label 20350 8600 0    50   ~ 0
 INT7_LATCH
+Text HLabel 8200 4300 0    50   Input ~ 0
+~INT0_OUT_NCLK
+Text HLabel 8200 4400 0    50   Input ~ 0
+~INT1_OUT_NCLK
+Text HLabel 8200 4500 0    50   Input ~ 0
+~INT2_OUT_NCLK
+Text HLabel 8200 4600 0    50   Input ~ 0
+~INT3_OUT_NCLK
+Text HLabel 8200 4700 0    50   Input ~ 0
+~INT4_OUT_NCLK
+Text HLabel 8200 4800 0    50   Input ~ 0
+~INT5_OUT_NCLK
+Text HLabel 8200 4900 0    50   Input ~ 0
+~INT6_OUT_NCLK
+Text HLabel 8200 5000 0    50   Input ~ 0
+~INT7_OUT_NCLK
+Text HLabel 20350 6450 2    50   Input ~ 0
+~INT0_OUT_NCLK
+Text HLabel 20350 6550 2    50   Input ~ 0
+~INT1_OUT_NCLK
+Text HLabel 20350 6650 2    50   Input ~ 0
+~INT2_OUT_NCLK
+Text HLabel 20350 6750 2    50   Input ~ 0
+~INT3_OUT_NCLK
+Text HLabel 20350 6850 2    50   Input ~ 0
+~INT4_OUT_NCLK
+Text HLabel 20350 6950 2    50   Input ~ 0
+~INT5_OUT_NCLK
+Text HLabel 20350 7050 2    50   Input ~ 0
+~INT6_OUT_NCLK
+Text HLabel 20350 7150 2    50   Input ~ 0
+~INT7_OUT_NCLK
+Text HLabel 18450 5350 0    50   Input ~ 0
+~PC0_IN_NCLK
+Text HLabel 18450 5450 0    50   Input ~ 0
+~PC1_IN_NCLK
+Text HLabel 18450 5550 0    50   Input ~ 0
+~PC2_IN_NCLK
 $EndSCHEMATC
