File: kicad/control_logic_leds.sch (KiCad schematic (older format))
At the start: 176 parts

Commit message: Going to try out resistor network.
Parts:
- added RN?: R_Network09, Resistor_THT:R_Array_SIP10, symbol Device:R_Network09
Changed lines of the file:
@@
 Text Notes 1650 1100 0    79   ~ 0
 IN plane
+$Comp
+L Device:R_Network09 RN?
+U 1 1 5B91DBAA
+P 3850 1750
+F 0 "RN?" V 3233 1750 50  0000 C CNN
+F 1 "R_Network09" V 3324 1750 50  0000 C CNN
+F 2 "Resistor_THT:R_Array_SIP10" V 4425 1750 50  0001 C CNN
+F 3 "http://www.vishay.com/docs/31509/csc.pdf" H 3850 1750 50  0001 C CNN
+	1    3850 1750
+	0    1    1    0
+$EndComp
 $EndSCHEMATC

Commit message: Change to resistor networks for LEDs.
Parts:
- removed R100, R101, R102, R103, R104, R105, R106, R107, R108, R109, R110, R111, R112, R113, R114, R115, R116, R117, R118, R119, R120, R121, R122, R17, R18, R19, R20, R21, R22, R41, R42, R43, R44, R45, R46, R47, R48, R49, R50, R51, R52, R53, R54, R55, R56, R57, R58, R59, R60, R61, R62, R63, R64, R65, R66, R67, R68, R69, R70, R71, R72, R73, R74, R75, R76, R77, R78, R79, R80, R81, R82, R83, R84, R85, R86, R87, R88, R89, R90, R91, R92, R93, R94, R95, R96, R97, R98, R99: 2.2K, Resistor_THT:R_Axial_DIN0207_L6.3mm_D2.5mm_P7.62mm_Horizontal, symbol Device:R
- added RN10, RN11, RN12, RN3, RN4, RN5, RN6, RN7, RN8, RN9: 2K, Resistor_THT:R_Array_SIP10, symbol Device:R_Network09
- RN2: renamed from RN?; value R_Network09 -> 2K
Connections:
- wire segments 176 -> 363
- no-connect marks 0 -> 11
Other:
- note added: "Control plane stuff"
- note added: "Interrupt stuff"
- note added: "TODO: replace bus with resistor network too."
- note removed: "Control plane"
- note removed: "Interrupt Related"

Commit message: Fix LEDs a bit.
Parts:
- removed RN7: 2K, Resistor_THT:R_Array_SIP10, symbol Device:R_Network09
Connections:
- net labels added: ~OPCODE0_IN, ~OPCODE1_IN, ~PC0_IN, ~PC1_IN, ~PC2_IN
- net labels removed: OPCODE0_IN, OPCODE1_IN, PC0_IN, PC1_IN, PC2_IN
- wire segments 363 -> 338
- no-connect marks 11 -> 2
