File: kicad/mlu.sch (KiCad schematic (older format))
At the start: 2 parts, among them U31 SST39SF040

Commit message: Schematic for kernel and user stack pointers.
Connections:
- net labels added: ~OUT
- net labels removed: OUT
Changed lines of the file:
@@
 $Descr A4 11693 8268
 encoding utf-8
-Sheet 15 17
+Sheet 15 19
 Title ""
 Date ""
@@
 B7
 Text HLabel 1350 3700 0    50   Input ~ 0
-OUT
+~OUT
 $Comp
 L power:GND #PWR0172
