File: kicad/clock.sch (KiCad schematic (older format))
At the start: 58 parts, among them SW1 SW_DIP_x03 - Clock Source Sel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, SW2 SW_Push, U1 LM555 - Adjustable Clock, U2 74HC14, U3 74151, U30 74HC86, U32 74LS107, U33 74LS08, U34 74LS107, U35 74LS107, U4 LM555 - Button Clock, U5 74HC04, U6 74LS138, Y1 12MHz

Commit message: Reset related progress.
Parts:
- added C?: 0.1uF, Capacitor_THT:C_Disc_D3.0mm_W2.0mm_P2.50mm, symbol Device:C_Small
- added R?: 100K, Resistor_THT:R_Axial_DIN0207_L6.3mm_D2.5mm_P7.62mm_Horizontal, symbol Device:R
- added R?: 1M, Resistor_THT:R_Axial_DIN0207_L6.3mm_D2.5mm_P7.62mm_Horizontal, symbol Device:R
- added SW?: SW_SPST, symbol Switch:SW_SPST
- added U117: 74LS08, symbol 74xx:74LS08
Connections:
- net labels added: ~RESET_NCLK
- wire segments 129 -> 135
Other:
- note added: "Clock Frontend"
- note added: "If either goes low (i.e. ~RESET),\nthen AND will go low."
- note added: "Reset Button"
- note added: "Spare AND taken \nfrom control logic"
- moved on the sheet: U2A, U2B, U2C, U2D, U2E, U2F, U2G, U30A, U30B, U30C, U30D, U30E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

Commit message: Small update.
Parts:
- gave numbers to parts that had none: 4
Changed lines of the file:
@@
 	1    0    0    -1
 $EndComp
-Wire Notes Line
-	14900 5600 14900 3700
-Text Notes 13800 4650 0    50   ~ 0
+Text Notes 13700 4950 0    50   ~ 0
 Spares
 Text HLabel 10250 5000 2    50   Input ~ 0
@@
 L power:GND #PWR0167
 U 1 1 5B0C83CD
-P 13100 4800
-F 0 "#PWR0167" H 13100 4550 50  0001 C CNN
-F 1 "GND" H 13105 4627 50  0000 C CNN
-F 2 "" H 13100 4800 50  0001 C CNN
-F 3 "" H 13100 4800 50  0001 C CNN
-	1    13100 4800
-	0    1    1    0
-$EndComp
-NoConn ~ 13700 4800
+P 14000 5250
+F 0 "#PWR0167" H 14000 5000 50  0001 C CNN
+F 1 "GND" H 14005 5077 50  0000 C CNN
+F 2 "" H 14000 5250 50  0001 C CNN
+F 3 "" H 14000 5250 50  0001 C CNN
+	1    14000 5250
+	0    1    1    0
+$EndComp
+NoConn ~ 14600 5250
 Text Notes 5450 5900 0    50   ~ 0
 Simulate a clock source change on\nreset to pull CLK low for a bit while\nmachine state is reset.
@@
 Clock Frontend
 $Comp
-L Switch:SW_SPST SW?
+L Switch:SW_SPST SW4
 U 1 1 5B386AD7
 P 5600 6850
-F 0 "SW?" V 5554 6948 50  0000 L CNN
+F 0 "SW4" V 5554 6948 50  0000 L CNN
 F 1 "SW_SPST" V 5645 6948 50  0000 L CNN
 F 2 "" H 5600 6850 50  0001 C CNN
@@
 Connection ~ 950  4550
 $Comp
-L Device:R R?
+L Device:R R15
 U 1 1 5B38C9B9
 P 5600 7550
-F 0 "R?" H 5670 7596 50  0000 L CNN
+F 0 "R15" H 5670 7596 50  0000 L CNN
 F 1 "100K" H 5670 7505 50  0000 L CNN
 F 2 "Resistor_THT:R_Axial_DIN0207_L6.3mm_D2.5mm_P7.62mm_Horizontal" V 5530 7550 50  0001 C CNN
@@
 	5600 7050 5600 7150
 $Comp
-L power:VCC #PWR?
+L power:VCC #PWR0126
 U 1 1 5B38C9C1
 P 5600 6650
-F 0 "#PWR?" H 5600 6500 50  0001 C CNN
+F 0 "#PWR0126" H 5600 6500 50  0001 C CNN
 F 1 "VCC" H 5617 6823 50  0000 C CNN
 F 2 "" H 5600 6650 50  0001 C CNN
@@
 $EndComp
 $Comp
-L Device:C_Small C?
+L Device:C_Small C114
 U 1 1 5B391B45
 P 6450 7250
-F 0 "C?" V 6221 7250 50  0000 C CNN
+F 0 "C114" V 6221 7250 50  0000 C CNN
 F 1 "0.1uF" V 6312 7250 50  0000 C CNN
 F 2 "Capacitor_THT:C_Disc_D3.0mm_W2.0mm_P2.50mm" H 6450 7250 50  0001 C CNN
@@
 $EndComp
 $Comp
-L power:GND #PWR?
+L power:GND #PWR0128
 U 1 1 5B391B4C
 P 6450 7350
-F 0 "#PWR?" H 6450 7100 50  0001 C CNN
+F 0 "#PWR0128" H 6450 7100 50  0001 C CNN
 F 1 "GND" H 6455 7177 50  0000 C CNN
 F 2 "" H 6450 7350 50  0001 C CNN
@@
 $EndComp
 $Comp
-L Device:R R?
+L Device:R R16
 U 1 1 5B391B52
 P 6100 7150
-F 0 "R?" V 5893 7150 50  0000 C CNN
+F 0 "R16" V 5893 7150 50  0000 C CNN
 F 1 "1M" V 5984 7150 50  0000 C CNN
 F 2 "Resistor_THT:R_Axial_DIN0207_L6.3mm_D2.5mm_P7.62mm_Horizontal" V 6030 7150 50  0001 C CNN
@@
 	5600 7150 5600 7400
 $Comp
-L power:GND #PWR?
+L power:GND #PWR0129
 U 1 1 5B39CA00
 P 5600 7700
-F 0 "#PWR?" H 5600 7450 50  0001 C CNN
+F 0 "#PWR0129" H 5600 7450 50  0001 C CNN
 F 1 "GND" H 5605 7527 50  0000 C CNN
 F 2 "" H 5600 7700 50  0001 C CNN

Commit message: Import into pcbnew.
Parts:
- removed SW4: SW_SPST, symbol Switch:SW_SPST
- added SW4: SW_Push, Button_Switch_THT:SW_PUSH_6mm_H7.3mm, symbol Switch:SW_Push
- U117: footprint (none) -> Package_DIP:DIP-14_W7.62mm_Socket
Changed lines of the file:
@@
 Text Notes 8950 3800 0    50   ~ 0
 Clock Frontend
-$Comp
-L Switch:SW_SPST SW4
-U 1 1 5B386AD7
-P 5600 6850
-F 0 "SW4" V 5554 6948 50  0000 L CNN
-F 1 "SW_SPST" V 5645 6948 50  0000 L CNN
-F 2 "" H 5600 6850 50  0001 C CNN
-F 3 "" H 5600 6850 50  0001 C CNN
-	1    5600 6850
-	0    1    1    0
-$EndComp
 Connection ~ 950  4550
 $Comp
@@
 F 0 "U117" H 8450 7575 50  0000 C CNN
 F 1 "74LS08" H 8450 7484 50  0000 C CNN
-F 2 "" H 8450 7250 50  0001 C CNN
+F 2 "Package_DIP:DIP-14_W7.62mm_Socket" H 8450 7250 50  0001 C CNN
 F 3 "http://www.ti.com/lit/gpn/sn74LS08" H 8450 7250 50  0001 C CNN
 	4    8450 7250
@@
 Text Notes 6700 6600 0    50   ~ 0
 Reset Button
+$Comp
+L Switch:SW_Push SW4
+U 1 1 5B1382CD
+P 5600 6850
+F 0 "SW4" H 5600 7135 50  0000 C CNN
+F 1 "SW_Push" H 5600 7044 50  0000 C CNN
+F 2 "Button_Switch_THT:SW_PUSH_6mm_H7.3mm" H 5600 7050 50  0001 C CNN
+F 3 "" H 5600 7050 50  0001 C CNN
+	1    5600 6850
+	0    -1   -1   0
+$EndComp
 $EndSCHEMATC

Commit message: Add control logic LEDs to schematic.
Parts:
- added unit 5 of U5
Connections:
- no-connect marks 9 -> 10
Changed lines of the file:
@@
 $Descr A3 16535 11693
 encoding utf-8
-Sheet 2 36
+Sheet 2 37
 Title ""
 Date ""
@@
 	0    -1   -1   0
 $EndComp
+$Comp
+L 74xx:74HC04 U5
+U 5 1 5B6B88E1
+P 14300 5750
+AR Path="/5ADF0E03/5B6B88E1" Ref="U5"  Part="5"
+AR Path="/5B6B88E1" Ref="U?"  Part="5"
+AR Path="/5B0C6DCD/5B6B88E1" Ref="U?"  Part="5"
+F 0 "U5" H 14300 6067 50  0000 C CNN
+F 1 "74HC04" H 14300 5976 50  0000 C CNN
+F 2 "Package_DIP:DIP-14_W7.62mm_Socket" H 14300 5750 50  0001 C CNN
+F 3 "http://www.nxp.com/documents/data_sheet/74HC_HCT04.pdf" H 14300 5750 50  0001 C CNN
+	5    14300 5750
+	1    0    0    -1
+$EndComp
+$Comp
+L power:GND #PWR0459
+U 1 1 5B6BDB28
+P 14000 5750
+F 0 "#PWR0459" H 14000 5500 50  0001 C CNN
+F 1 "GND" H 14005 5577 50  0000 C CNN
+F 2 "" H 14000 5750 50  0001 C CNN
+F 3 "" H 14000 5750 50  0001 C CNN
+	1    14000 5750
+	0    1    1    0
+$EndComp
+NoConn ~ 14600 5750
 $EndSCHEMATC

Commit message: Small layout changes.
Parts:
- R2: footprint Potentiometer_THT:Potentiometer_Omeg_PC16BU_Vertical -> cpu:Akizuki-Denshi Potentiometer
Changed lines of the file:
@@
 F 0 "R2" H 2878 1646 50  0000 L CNN
 F 1 "1M" H 2878 1555 50  0000 L CNN
-F 2 "Potentiometer_THT:Potentiometer_Omeg_PC16BU_Vertical" V 2680 1600 50  0001 C CNN
+F 2 "cpu:Akizuki-Denshi Potentiometer" V 2680 1600 50  0001 C CNN
 F 3 "~" H 2750 1600 50  0001 C CNN
 	1    2750 1600

Commit message: Layout progress.
Parts:
- added C135: 0.1uF, Capacitor_THT:C_Disc_D3.0mm_W2.0mm_P2.50mm, symbol Device:C_Small
Connections:
- wire segments 135 -> 136
Changed lines of the file:
@@
 $EndComp
 NoConn ~ 14600 5750
+$Comp
+L Device:C_Small C135
+U 1 1 5B194605
+P 3200 5650
+F 0 "C135" H 3292 5696 50  0000 L CNN
+F 1 "0.1uF" H 3292 5605 50  0000 L CNN
+F 2 "Capacitor_THT:C_Disc_D3.0mm_W2.0mm_P2.50mm" H 3200 5650 50  0001 C CNN
+F 3 "~" H 3200 5650 50  0001 C CNN
+	1    3200 5650
+	1    0    0    1
+$EndComp
+Wire Wire Line
+	3650 5750 3200 5750
+Connection ~ 3650 5750
+$Comp
+L power:GND #PWR0460
+U 1 1 5B199E40
+P 3200 5550
+F 0 "#PWR0460" H 3200 5300 50  0001 C CNN
+F 1 "GND" H 3205 5377 50  0000 C CNN
+F 2 "" H 3200 5550 50  0001 C CNN
+F 3 "" H 3200 5550 50  0001 C CNN
+	1    3200 5550
+	0    1    1    0
+$EndComp
 $EndSCHEMATC

Commit message: Removed LEDs. Layout changes.
Connections:
- net labels removed: LED_VCC
Changed lines of the file:
@@
 $Descr A3 16535 11693
 encoding utf-8
-Sheet 2 37
+Sheet 2 35
 Title ""
 Date ""
@@
 Wire Wire Line
 	4450 6750 4650 6750
-Text GLabel 4650 5500 0    50   Input ~ 0
-LED_VCC
 $Comp
 L Device:LED D2
@@
 	0    1    1    0
 $EndComp
+$Comp
+L power:VCC #PWR0139
+U 1 1 5B1D0221
+P 4650 5500
+F 0 "#PWR0139" H 4650 5350 50  0001 C CNN
+F 1 "VCC" H 4667 5673 50  0000 C CNN
+F 2 "" H 4650 5500 50  0001 C CNN
+F 3 "" H 4650 5500 50  0001 C CNN
+	1    4650 5500
+	1    0    0    -1
+$EndComp
 $EndSCHEMATC
