File: kicad/5_32_decoder.sch (KiCad schematic (older format))
At the start: 4 parts, among them U93 74LS154, U94 74LS154

Commit message: Update layout with new capacitor sizes, etc.
Parts:
- C104, C105: footprint Capacitor_THT:C_Disc_D3.0mm_W2.0mm_P2.50mm -> Capacitor_THT:C_Disc_D6.0mm_W2.5mm_P5.00mm
Changed lines of the file:
@@
 F 0 "C106" V 1671 950 50  0000 C CNN
 F 1 "0.1uF" V 1762 950 50  0000 C CNN
-F 2 "Capacitor_THT:C_Disc_D3.0mm_W2.0mm_P2.50mm" H 1900 950 50  0001 C CNN
+F 2 "Capacitor_THT:C_Disc_D6.0mm_W2.5mm_P5.00mm" H 1900 950 50  0001 C CNN
 F 3 "~" H 1900 950 50  0001 C CNN
 	1    1900 950
@@
 F 0 "C107" V 3371 950 50  0000 C CNN
 F 1 "0.1uF" V 3462 950 50  0000 C CNN
-F 2 "Capacitor_THT:C_Disc_D3.0mm_W2.0mm_P2.50mm" H 3600 950 50  0001 C CNN
+F 2 "Capacitor_THT:C_Disc_D6.0mm_W2.5mm_P5.00mm" H 3600 950 50  0001 C CNN
 F 3 "~" H 3600 950 50  0001 C CNN
 	1    3600 950
