File: kicad/display_module.sch (KiCad schematic (older format))
At the start: 25 parts, among them SW5 SW_DIP_x03, U21 LM555, U22 74LS107, U23 74LS139, U24 AT28C64B, U25 HDSP-7803, U26 HDSP-7803, U27 HDSP-7803, U28 HDSP-7803

Commit message: Layout progress.
Connections:
- net labels removed: CARRY
Changed lines of the file:
@@
 Text Label 5500 2300 2    50   ~ 0
 DISP_CLK
-Text Label 5500 2400 2    50   ~ 0
-CARRY
 $Comp
 L 74xx:74LS139 U23
@@
 	0    -1   -1   0
 $EndComp
+Text Label 5500 2400 2    50   ~ 0
+C0
 $EndSCHEMATC

Commit message: Layout progress.
Parts:
- removed C31: 1uF, Capacitor_THT:CP_Radial_D5.0mm_P2.50mm, symbol Device:C_Small
Connections:
- wire segments 59 -> 57
Changed lines of the file:
@@
-$EndComp
-$Comp
-L Device:C_Small C31
-U 1 1 5AFEE817
-P 3050 1300
-F 0 "C31" H 3142 1346 50  0000 L CNN
-F 1 "1uF" H 3142 1255 50  0000 L CNN
-F 2 "Capacitor_THT:CP_Radial_D5.0mm_P2.50mm" H 3050 1300 50  0001 C CNN
-F 3 "~" H 3050 1300 50  0001 C CNN
-	1    3050 1300
-	1    0    0    -1
 $EndComp
 $Comp
@@
 	1    0    0    -1
 $EndComp
-Wire Wire Line
-	3350 1600 3050 1600
-Wire Wire Line
-	3050 1600 3050 1400
 Connection ~ 3350 1600
 Wire Wire Line
@@
 	3550 1600 3550 1400
 $Comp
-L power:GND #PWR0139
-U 1 1 5AFEF443
-P 3050 1200
-F 0 "#PWR0139" H 3050 950 50  0001 C CNN
-F 1 "GND" V 3055 1072 50  0000 R CNN
-F 2 "" H 3050 1200 50  0001 C CNN
-F 3 "" H 3050 1200 50  0001 C CNN
-	1    3050 1200
-	0    1    1    0
-$EndComp
-$Comp
 L power:GND #PWR0140

Commit message: Update layout with new capacitor sizes, etc.
Parts:
- C29: footprint Capacitor_THT:C_Disc_D3.0mm_W2.0mm_P2.50mm -> Capacitor_THT:C_Disc_D5.0mm_W2.5mm_P5.00mm
- C30, C32, C33, C34, C35: footprint Capacitor_THT:C_Disc_D3.0mm_W2.0mm_P2.50mm -> Capacitor_THT:C_Disc_D6.0mm_W2.5mm_P5.00mm
Changed lines of the file:
@@
 F 0 "C32" H 3642 1346 50  0000 L CNN
 F 1 "0.1uF" H 3642 1255 50  0000 L CNN
-F 2 "Capacitor_THT:C_Disc_D3.0mm_W2.0mm_P2.50mm" H 3550 1300 50  0001 C CNN
+F 2 "Capacitor_THT:C_Disc_D6.0mm_W2.5mm_P5.00mm" H 3550 1300 50  0001 C CNN
 F 3 "~" H 3550 1300 50  0001 C CNN
 	1    3550 1300
@@
 F 0 "C29" H 2342 2146 50  0000 L CNN
 F 1 "10nF" H 2342 2055 50  0000 L CNN
-F 2 "Capacitor_THT:C_Disc_D3.0mm_W2.0mm_P2.50mm" H 2250 2100 50  0001 C CNN
+F 2 "Capacitor_THT:C_Disc_D5.0mm_W2.5mm_P5.00mm" H 2250 2100 50  0001 C CNN
 F 3 "~" H 2250 2100 50  0001 C CNN
 	1    2250 2100
@@
 F 0 "C30" V 2371 1800 50  0000 C CNN
 F 1 "0.1nF" V 2462 1800 50  0000 C CNN
-F 2 "Capacitor_THT:C_Disc_D3.0mm_W2.0mm_P2.50mm" H 2600 1800 50  0001 C CNN
+F 2 "Capacitor_THT:C_Disc_D6.0mm_W2.5mm_P5.00mm" H 2600 1800 50  0001 C CNN
 F 3 "~" H 2600 1800 50  0001 C CNN
 	1    2600 1800
@@
 F 0 "C33" V 4671 550 50  0000 C CNN
 F 1 "0.1uF" V 4762 550 50  0000 C CNN
-F 2 "Capacitor_THT:C_Disc_D3.0mm_W2.0mm_P2.50mm" H 4900 550 50  0001 C CNN
+F 2 "Capacitor_THT:C_Disc_D6.0mm_W2.5mm_P5.00mm" H 4900 550 50  0001 C CNN
 F 3 "~" H 4900 550 50  0001 C CNN
 	1    4900 550
@@
 F 0 "C34" V 6871 450 50  0000 C CNN
 F 1 "0.1uF" V 6962 450 50  0000 C CNN
-F 2 "Capacitor_THT:C_Disc_D3.0mm_W2.0mm_P2.50mm" H 7100 450 50  0001 C CNN
+F 2 "Capacitor_THT:C_Disc_D6.0mm_W2.5mm_P5.00mm" H 7100 450 50  0001 C CNN
 F 3 "~" H 7100 450 50  0001 C CNN
 	1    7100 450
@@
 F 0 "C35" H 8258 4354 50  0000 R CNN
 F 1 "0.1uF" H 8258 4445 50  0000 R CNN
-F 2 "Capacitor_THT:C_Disc_D3.0mm_W2.0mm_P2.50mm" H 8350 4400 50  0001 C CNN
+F 2 "Capacitor_THT:C_Disc_D6.0mm_W2.5mm_P5.00mm" H 8350 4400 50  0001 C CNN
 F 3 "~" H 8350 4400 50  0001 C CNN
 	1    8350 4400
