File: kicad/flag_logic.sch (KiCad schematic (older format))
At the start: 4 parts, among them U119 74LS32, U120 74LS32

Commit message: Import into pcbnew.
Parts:
- C130, C131: value C_Small -> 0.1uF; footprint (none) -> Capacitor_THT:C_Disc_D3.0mm_W2.0mm_P2.50mm
- U119, U120: footprint (none) -> Package_DIP:DIP-14_W7.62mm_Socket
Changed lines of the file:
@@
 F 0 "U119" H 1200 1675 50  0000 C CNN
 F 1 "74LS32" H 1200 1584 50  0000 C CNN
-F 2 "" H 1200 1350 50  0001 C CNN
+F 2 "Package_DIP:DIP-14_W7.62mm_Socket" H 1200 1350 50  0001 C CNN
 F 3 "http://www.ti.com/lit/gpn/sn74LS32" H 1200 1350 50  0001 C CNN
 	1    1200 1350
@@
 F 0 "U119" H 1200 2225 50  0000 C CNN
 F 1 "74LS32" H 1200 2134 50  0000 C CNN
-F 2 "" H 1200 1900 50  0001 C CNN
+F 2 "Package_DIP:DIP-14_W7.62mm_Socket" H 1200 1900 50  0001 C CNN
 F 3 "http://www.ti.com/lit/gpn/sn74LS32" H 1200 1900 50  0001 C CNN
 	2    1200 1900
@@
 F 0 "U119" H 1200 2775 50  0000 C CNN
 F 1 "74LS32" H 1200 2684 50  0000 C CNN
-F 2 "" H 1200 2450 50  0001 C CNN
+F 2 "Package_DIP:DIP-14_W7.62mm_Socket" H 1200 2450 50  0001 C CNN
 F 3 "http://www.ti.com/lit/gpn/sn74LS32" H 1200 2450 50  0001 C CNN
 	3    1200 2450
@@
 F 0 "U119" H 1200 3325 50  0000 C CNN
 F 1 "74LS32" H 1200 3234 50  0000 C CNN
-F 2 "" H 1200 3000 50  0001 C CNN
+F 2 "Package_DIP:DIP-14_W7.62mm_Socket" H 1200 3000 50  0001 C CNN
 F 3 "http://www.ti.com/lit/gpn/sn74LS32" H 1200 3000 50  0001 C CNN
 	4    1200 3000
@@
 F 0 "U119" V 1233 700 50  0000 C CNN
 F 1 "74LS32" V 1324 700 50  0000 C CNN
-F 2 "" H 1600 700 50  0001 C CNN
+F 2 "Package_DIP:DIP-14_W7.62mm_Socket" H 1600 700 50  0001 C CNN
 F 3 "http://www.ti.com/lit/gpn/sn74LS32" H 1600 700 50  0001 C CNN
 	5    1600 700
@@
 P 2100 600
 F 0 "C130" H 2192 646 50  0000 L CNN
-F 1 "C_Small" H 2192 555 50  0000 L CNN
-F 2 "" H 2100 600 50  0001 C CNN
+F 1 "0.1uF" H 2192 555 50  0000 L CNN
+F 2 "Capacitor_THT:C_Disc_D3.0mm_W2.0mm_P2.50mm" H 2100 600 50  0001 C CNN
 F 3 "~" H 2100 600 50  0001 C CNN
 	1    2100 600
@@
 F 0 "U120" H 2150 1925 50  0000 C CNN
 F 1 "74LS32" H 2150 1834 50  0000 C CNN
-F 2 "" H 2150 1600 50  0001 C CNN
+F 2 "Package_DIP:DIP-14_W7.62mm_Socket" H 2150 1600 50  0001 C CNN
 F 3 "http://www.ti.com/lit/gpn/sn74LS32" H 2150 1600 50  0001 C CNN
 	1    2150 1600
@@
 F 0 "U120" H 2200 3025 50  0000 C CNN
 F 1 "74LS32" H 2200 2934 50  0000 C CNN
-F 2 "" H 2200 2700 50  0001 C CNN
+F 2 "Package_DIP:DIP-14_W7.62mm_Socket" H 2200 2700 50  0001 C CNN
 F 3 "http://www.ti.com/lit/gpn/sn74LS32" H 2200 2700 50  0001 C CNN
 	2    2200 2700
@@
 F 0 "U120" H 2950 2425 50  0000 C CNN
 F 1 "74LS32" H 2950 2334 50  0000 C CNN
-F 2 "" H 2950 2100 50  0001 C CNN
+F 2 "Package_DIP:DIP-14_W7.62mm_Socket" H 2950 2100 50  0001 C CNN
 F 3 "http://www.ti.com/lit/gpn/sn74LS32" H 2950 2100 50  0001 C CNN
 	3    2950 2100
@@
 F 0 "U120" H 1800 3925 50  0000 C CNN
 F 1 "74LS32" H 1800 3834 50  0000 C CNN
-F 2 "" H 1800 3600 50  0001 C CNN
+F 2 "Package_DIP:DIP-14_W7.62mm_Socket" H 1800 3600 50  0001 C CNN
 F 3 "http://www.ti.com/lit/gpn/sn74LS32" H 1800 3600 50  0001 C CNN
 	4    1800 3600
@@
 F 0 "U120" V 2983 850 50  0000 C CNN
 F 1 "74LS32" V 3074 850 50  0000 C CNN
-F 2 "" H 3350 850 50  0001 C CNN
+F 2 "Package_DIP:DIP-14_W7.62mm_Socket" H 3350 850 50  0001 C CNN
 F 3 "http://www.ti.com/lit/gpn/sn74LS32" H 3350 850 50  0001 C CNN
 	5    3350 850
@@
 P 3850 750
 F 0 "C131" H 3942 796 50  0000 L CNN
-F 1 "C_Small" H 3942 705 50  0000 L CNN
-F 2 "" H 3850 750 50  0001 C CNN
+F 1 "0.1uF" H 3942 705 50  0000 L CNN
+F 2 "Capacitor_THT:C_Disc_D3.0mm_W2.0mm_P2.50mm" H 3850 750 50  0001 C CNN
 F 3 "~" H 3850 750 50  0001 C CNN
 	1    3850 750

Commit message: Update layout with new capacitor sizes, etc.
Parts:
- C130, C131: footprint Capacitor_THT:C_Disc_D3.0mm_W2.0mm_P2.50mm -> Capacitor_THT:C_Disc_D6.0mm_W2.5mm_P5.00mm
Changed lines of the file:
@@
 F 0 "C130" H 2192 646 50  0000 L CNN
 F 1 "0.1uF" H 2192 555 50  0000 L CNN
-F 2 "Capacitor_THT:C_Disc_D3.0mm_W2.0mm_P2.50mm" H 2100 600 50  0001 C CNN
+F 2 "Capacitor_THT:C_Disc_D6.0mm_W2.5mm_P5.00mm" H 2100 600 50  0001 C CNN
 F 3 "~" H 2100 600 50  0001 C CNN
 	1    2100 600
@@
 F 0 "C131" H 3942 796 50  0000 L CNN
 F 1 "0.1uF" H 3942 705 50  0000 L CNN
-F 2 "Capacitor_THT:C_Disc_D3.0mm_W2.0mm_P2.50mm" H 3850 750 50  0001 C CNN
+F 2 "Capacitor_THT:C_Disc_D6.0mm_W2.5mm_P5.00mm" H 3850 750 50  0001 C CNN
 F 3 "~" H 3850 750 50  0001 C CNN
 	1    3850 750
