File: kicad/microop_counter.sch (KiCad schematic (older format))
At the start: 2 parts, among them U107 74LS161

Commit message: Reset related progress.
Connections:
- net labels added: CLK
- net labels removed: ~CLK
Changed lines of the file:
@@
 $Descr A4 11693 8268
 encoding utf-8
-Sheet 36 36
+Sheet 30 36
 Title ""
 Date ""
@@
 ~RESET
 Text HLabel 1250 2100 0    50   Input ~ 0
-~CLK
+CLK
 $Comp
 L power:VCC #PWR037

Commit message: Update layout with new capacitor sizes, etc.
Parts:
- C118: footprint Capacitor_THT:C_Disc_D3.0mm_W2.0mm_P2.50mm -> Capacitor_THT:C_Disc_D6.0mm_W2.5mm_P5.00mm
Changed lines of the file:
@@
 F 0 "C118" V 1821 1000 50  0000 C CNN
 F 1 "0.1uF" V 1912 1000 50  0000 C CNN
-F 2 "Capacitor_THT:C_Disc_D3.0mm_W2.0mm_P2.50mm" H 2050 1000 50  0001 C CNN
+F 2 "Capacitor_THT:C_Disc_D6.0mm_W2.5mm_P5.00mm" H 2050 1000 50  0001 C CNN
 F 3 "~" H 2050 1000 50  0001 C CNN
 	1    2050 1000
