File: kicad/opcode_register.sch (KiCad schematic (older format))
At the start: 6 parts, among them U105 74LS161, U106 74LS161, U91 74LS161

Commit message: Update layout with new capacitor sizes, etc.
Parts:
- C103, C116, C117: footprint Capacitor_THT:C_Disc_D3.0mm_W2.0mm_P2.50mm -> Capacitor_THT:C_Disc_D6.0mm_W2.5mm_P5.00mm
Changed lines of the file:
@@
 F 0 "C103" V 1821 800 50  0000 C CNN
 F 1 "0.1uF" V 1912 800 50  0000 C CNN
-F 2 "Capacitor_THT:C_Disc_D3.0mm_W2.0mm_P2.50mm" H 2050 800 50  0001 C CNN
+F 2 "Capacitor_THT:C_Disc_D6.0mm_W2.5mm_P5.00mm" H 2050 800 50  0001 C CNN
 F 3 "~" H 2050 800 50  0001 C CNN
 	1    2050 800
@@
 F 0 "C117" V 3671 800 50  0000 C CNN
 F 1 "0.1uF" V 3762 800 50  0000 C CNN
-F 2 "Capacitor_THT:C_Disc_D3.0mm_W2.0mm_P2.50mm" H 3900 800 50  0001 C CNN
+F 2 "Capacitor_THT:C_Disc_D6.0mm_W2.5mm_P5.00mm" H 3900 800 50  0001 C CNN
 F 3 "~" H 3900 800 50  0001 C CNN
 	1    3900 800
@@
 F 0 "C116" V 2171 3300 50  0000 C CNN
 F 1 "0.1uF" V 2262 3300 50  0000 C CNN
-F 2 "Capacitor_THT:C_Disc_D3.0mm_W2.0mm_P2.50mm" H 2400 3300 50  0001 C CNN
+F 2 "Capacitor_THT:C_Disc_D6.0mm_W2.5mm_P5.00mm" H 2400 3300 50  0001 C CNN
 F 3 "~" H 2400 3300 50  0001 C CNN
 	1    2400 3300
