File: eeprom_programmer/pcb/eeprom_programmer.sch (KiCad schematic (older format))
At the start: 12 parts, among them SW1 SW_DIP_x03, U1 74HC595, U2 74HC595, U3 74HC595, U4 SST39SF040, U5 AT28C64B

Commit message: Update layout with new capacitor sizes, etc.
Parts:
- U1, U2, U3: symbol 74xx:74HC595 -> eeprom_programmer-rescue:74HC595-74xx
Changed lines of the file:
@@
 $EndComp
 $Comp
-L 74xx:74HC595 U1
+L eeprom_programmer-rescue:74HC595-74xx U1
 U 1 1 5AD2D7E6
 P 1300 1600
@@
 $EndComp
 $Comp
-L 74xx:74HC595 U2
+L eeprom_programmer-rescue:74HC595-74xx U2
 U 1 1 5AD2D89E
 P 2850 1600
@@
 $EndComp
 $Comp
-L 74xx:74HC595 U3
+L eeprom_programmer-rescue:74HC595-74xx U3
 U 1 1 5AD2D95A
 P 4350 1600

Commit message: Fix arduino d13 LED pullup bug.
Parts:
- added R3: 100K, Resistor_THT:R_Axial_DIN0207_L6.3mm_D2.5mm_P7.62mm_Horizontal, symbol Device:R
- U1, U2, U3: symbol eeprom_programmer-rescue:74HC595-74xx -> eeprom_programmer-rescue:74HC595-74xx-eeprom_programmer-rescue
Connections:
- wire segments 22 -> 19
Other:
- note added: "Use internal pullups on D11 and D12.\nUse external pull-down on D13\nbecause of attached LED."
Changed lines of the file:
@@
 $EndComp
 $Comp
-L eeprom_programmer-rescue:74HC595-74xx U1
+L eeprom_programmer-rescue:74HC595-74xx-eeprom_programmer-rescue U1
 U 1 1 5AD2D7E6
 P 1300 1600
@@
 $EndComp
 $Comp
-L eeprom_programmer-rescue:74HC595-74xx U2
+L eeprom_programmer-rescue:74HC595-74xx-eeprom_programmer-rescue U2
 U 1 1 5AD2D89E
 P 2850 1600
@@
 $EndComp
 $Comp
-L eeprom_programmer-rescue:74HC595-74xx U3
+L eeprom_programmer-rescue:74HC595-74xx-eeprom_programmer-rescue U3
 U 1 1 5AD2D95A
 P 4350 1600
@@
 L Switch:SW_DIP_x03 SW1
 U 1 1 5AF911FD
-P 1450 6000
-F 0 "SW1" V 1404 6330 50  0000 L CNN
-F 1 "SW_DIP_x03" V 1495 6330 50  0000 L CNN
-F 2 "Button_Switch_THT:SW_DIP_SPSTx03_Slide_9.78x9.8mm_W7.62mm_P2.54mm" H 1450 6000 50  0001 C CNN
-F 3 "" H 1450 6000 50  0001 C CNN
-	1    1450 6000
+P 1300 6350
+F 0 "SW1" V 1254 6680 50  0000 L CNN
+F 1 "SW_DIP_x03" V 1345 6680 50  0000 L CNN
+F 2 "Button_Switch_THT:SW_DIP_SPSTx03_Slide_9.78x9.8mm_W7.62mm_P2.54mm" H 1300 6350 50  0001 C CNN
+F 3 "" H 1300 6350 50  0001 C CNN
+	1    1300 6350
 	0    1    1    0
 $EndComp
 Wire Wire Line
 	1450 4750 1300 4750
-Wire Wire Line
-	1300 4750 1300 5700
-Wire Wire Line
-	1300 5700 1450 5700
-Wire Wire Line
-	1450 4850 1350 4850
-Wire Wire Line
-	1350 4850 1350 5600
-Wire Wire Line
-	1350 5600 1550 5600
-Wire Wire Line
-	1550 5600 1550 5700
-Wire Wire Line
-	1450 4950 1450 5500
-Wire Wire Line
-	1450 5500 1650 5500
-Wire Wire Line
-	1650 5500 1650 5700
 $Comp
 L power:GND #PWR0126
 U 1 1 5AF916B7
-P 1450 6300
-F 0 "#PWR0126" H 1450 6050 50  0001 C CNN
-F 1 "GND" H 1455 6127 50  0000 C CNN
-F 2 "" H 1450 6300 50  0001 C CNN
-F 3 "" H 1450 6300 50  0001 C CNN
-	1    1450 6300
-	1    0    0    -1
-$EndComp
-Wire Wire Line
-	1650 6300 1550 6300
-Wire Wire Line
-	1550 6300 1450 6300
-Connection ~ 1550 6300
-Connection ~ 1450 6300
+P 1300 6650
+F 0 "#PWR0126" H 1300 6400 50  0001 C CNN
+F 1 "GND" H 1305 6477 50  0000 C CNN
+F 2 "" H 1300 6650 50  0001 C CNN
+F 3 "" H 1300 6650 50  0001 C CNN
+	1    1300 6650
+	1    0    0    -1
+$EndComp
+Wire Wire Line
+	1400 6650 1300 6650
+Wire Wire Line
+	1300 4750 1300 6050
+Wire Wire Line
+	1450 4850 1400 4850
+Wire Wire Line
+	1400 4850 1400 6050
+Wire Wire Line
+	1450 4950 1450 5800
+Wire Wire Line
+	1450 6050 1500 6050
+Connection ~ 1300 6650
+$Comp
+L power:+5V #PWR0127
+U 1 1 5B325FE8
+P 1500 6650
+F 0 "#PWR0127" H 1500 6500 50  0001 C CNN
+F 1 "+5V" V 1515 6778 50  0000 L CNN
+F 2 "" H 1500 6650 50  0001 C CNN
+F 3 "" H 1500 6650 50  0001 C CNN
+	1    1500 6650
+	-1   0    0    1
+$EndComp
+Text Notes 2250 6200 0    50   ~ 0
+Use internal pullups on D11 and D12.\nUse external pull-down on D13\nbecause of attached LED.
+$Comp
+L Device:R R3
+U 1 1 5B3266A6
+P 1900 5800
+F 0 "R3" V 1693 5800 50  0000 C CNN
+F 1 "100K" V 1784 5800 50  0000 C CNN
+F 2 "Resistor_THT:R_Axial_DIN0207_L6.3mm_D2.5mm_P7.62mm_Horizontal" V 1830 5800 50  0001 C CNN
+F 3 "~" H 1900 5800 50  0001 C CNN
+	1    1900 5800
+	0    1    1    0
+$EndComp
+$Comp
+L power:GND #PWR0128
+U 1 1 5B326728
+P 2050 5800
+F 0 "#PWR0128" H 2050 5550 50  0001 C CNN
+F 1 "GND" H 2055 5627 50  0000 C CNN
+F 2 "" H 2050 5800 50  0001 C CNN
+F 3 "" H 2050 5800 50  0001 C CNN
+	1    2050 5800
+	0    -1   -1   0
+$EndComp
+Wire Wire Line
+	1750 5800 1450 5800
+Connection ~ 1450 5800
+Wire Wire Line
+	1450 5800 1450 6050
 $EndSCHEMATC

Commit message: Update symbol in EEPROM pcb.
Parts:
- removed U1, U2, U3: 74HC595, Package_DIP:DIP-16_W7.62mm_Socket, symbol eeprom_programmer-rescue:74HC595-74xx-eeprom_programmer-rescue
- added U1, U2, U3: 74HC595, symbol 74xx:74HC595
Changed lines of the file:
@@
-$EndComp
-$Comp
-L eeprom_programmer-rescue:74HC595-74xx-eeprom_programmer-rescue U1
-U 1 1 5AD2D7E6
-P 1300 1600
-F 0 "U1" H 1300 2478 50  0000 C CNN
-F 1 "74HC595" H 1300 2387 50  0000 C CNN
-F 2 "Package_DIP:DIP-16_W7.62mm_Socket" H 1300 1600 50  0001 C CNN
-F 3 "http://www.nxp.com/documents/data_sheet/74HC_HCT595.pdf" H 1300 1600 50  0001 C CNN
-	1    1300 1600
-	1    0    0    -1
-$EndComp
-$Comp
-L eeprom_programmer-rescue:74HC595-74xx-eeprom_programmer-rescue U2
-U 1 1 5AD2D89E
-P 2850 1600
-F 0 "U2" H 2850 2478 50  0000 C CNN
-F 1 "74HC595" H 2850 2387 50  0000 C CNN
-F 2 "Package_DIP:DIP-16_W7.62mm_Socket" H 2850 1600 50  0001 C CNN
-F 3 "http://www.nxp.com/documents/data_sheet/74HC_HCT595.pdf" H 2850 1600 50  0001 C CNN
-	1    2850 1600
-	1    0    0    -1
-$EndComp
-$Comp
-L eeprom_programmer-rescue:74HC595-74xx-eeprom_programmer-rescue U3
-U 1 1 5AD2D95A
-P 4350 1600
-F 0 "U3" H 4350 2478 50  0000 C CNN
-F 1 "74HC595" H 4350 2387 50  0000 C CNN
-F 2 "Package_DIP:DIP-16_W7.62mm_Socket" H 4350 1600 50  0001 C CNN
-F 3 "http://www.nxp.com/documents/data_sheet/74HC_HCT595.pdf" H 4350 1600 50  0001 C CNN
-	1    4350 1600
-	1    0    0    -1
 $EndComp
 $Comp
@@
 NoConn ~ 2450 4950
 NoConn ~ 2450 4050
-Text Label 1800 1200 0    50   ~ 0
+Text Label 1700 1100 0    50   ~ 0
 A0
-Text Label 1800 1300 0    50   ~ 0
+Text Label 1700 1200 0    50   ~ 0
 A1
-Text Label 1800 1400 0    50   ~ 0
+Text Label 1700 1300 0    50   ~ 0
 A2
-Text Label 1800 1500 0    50   ~ 0
+Text Label 1700 1400 0    50   ~ 0
 A3
-Text Label 1800 1600 0    50   ~ 0
+Text Label 1700 1500 0    50   ~ 0
 A4
-Text Label 1800 1700 0    50   ~ 0
+Text Label 1700 1600 0    50   ~ 0
 A5
-Text Label 1800 1800 0    50   ~ 0
+Text Label 1700 1700 0    50   ~ 0
 A6
-Text Label 1800 1900 0    50   ~ 0
+Text Label 1700 1800 0    50   ~ 0
 A7
-Text Label 3350 1200 0    50   ~ 0
+Text Label 3250 1100 0    50   ~ 0
 A8
-Text Label 3350 1300 0    50   ~ 0
+Text Label 3250 1200 0    50   ~ 0
 A9
-Text Label 3350 1400 0    50   ~ 0
+Text Label 3250 1300 0    50   ~ 0
 A10
-Text Label 3350 1500 0    50   ~ 0
+Text Label 3250 1400 0    50   ~ 0
 A11
-Text Label 3350 1600 0    50   ~ 0
+Text Label 3250 1500 0    50   ~ 0
 A12
-Text Label 3350 1700 0    50   ~ 0
+Text Label 3250 1600 0    50   ~ 0
 A13
-Text Label 3350 1800 0    50   ~ 0
+Text Label 3250 1700 0    50   ~ 0
 A14
-Text Label 3350 1900 0    50   ~ 0
+Text Label 3250 1800 0    50   ~ 0
 A15
-Text Label 4850 1200 0    50   ~ 0
+Text Label 4750 1100 0    50   ~ 0
 A16
-Text Label 4850 1300 0    50   ~ 0
+Text Label 4750 1200 0    50   ~ 0
 A17
-Text Label 4850 1400 0    50   ~ 0
+Text Label 4750 1300 0    50   ~ 0
 A18
-NoConn ~ 4850 2100
+NoConn ~ 4750 2000
 Text Label 3100 3100 2    50   ~ 0
 A0
@@
 $EndComp
 Wire Wire Line
-	1800 2100 2150 2100
-Wire Wire Line
-	2150 2100 2150 1200
-Wire Wire Line
-	2150 1200 2350 1200
-Wire Wire Line
-	3350 2100 3600 2100
-Wire Wire Line
-	3600 2100 3600 1200
-Wire Wire Line
-	3600 1200 3850 1200
+	1950 2000 1950 1100
+Wire Wire Line
+	3250 2000 3500 2000
+Wire Wire Line
+	3500 2000 3500 1100
 $Comp
 L power:+5V #PWR0101
 U 1 1 5AD320D1
-P 3850 1500
-F 0 "#PWR0101" H 3850 1350 50  0001 C CNN
-F 1 "+5V" V 3865 1628 50  0000 L CNN
-F 2 "" H 3850 1500 50  0001 C CNN
-F 3 "" H 3850 1500 50  0001 C CNN
-	1    3850 1500
+P 3950 1400
+F 0 "#PWR0101" H 3950 1250 50  0001 C CNN
+F 1 "+5V" V 3965 1528 50  0000 L CNN
+F 2 "" H 3950 1400 50  0001 C CNN
+F 3 "" H 3950 1400 50  0001 C CNN
+	1    3950 1400
 	0    -1   -1   0
 $EndComp
@@
 L power:+5V #PWR0102
 U 1 1 5AD3211A
-P 2350 1500
-F 0 "#PWR0102" H 2350 1350 50  0001 C CNN
-F 1 "+5V" V 2365 1628 50  0000 L CNN
-F 2 "" H 2350 1500 50  0001 C CNN
-F 3 "" H 2350 1500 50  0001 C CNN
-	1    2350 1500
+P 2450 1400
+F 0 "#PWR0102" H 2450 1250 50  0001 C CNN
+F 1 "+5V" V 2465 1528 50  0000 L CNN
+F 2 "" H 2450 1400 50  0001 C CNN
+F 3 "" H 2450 1400 50  0001 C CNN
+	1    2450 1400
 	0    -1   -1   0
 $EndComp
@@
 Text Label 800  1400 2    50   ~ 0
 SRCLK
-Text Label 2350 1400 2    50   ~ 0
+Text Label 2450 1300 2    50   ~ 0
 SRCLK
-Text Label 3850 1400 2    50   ~ 0
+Text Label 3950 1300 2    50   ~ 0
 SRCLK
 Text Label 1450 4050 2    50   ~ 0
@@
 Text Label 800  1700 2    50   ~ 0
 RCLK
-Text Label 2350 1700 2    50   ~ 0
+Text Label 2450 1600 2    50   ~ 0
 RCLK
-Text Label 3850 1700 2    50   ~ 0
+Text Label 3950 1600 2    50   ~ 0
 RCLK
 $Comp
@@
 L power:GND #PWR0105
 U 1 1 5AD32457
-P 2350 1800
-F 0 "#PWR0105" H 2350 1550 50  0001 C CNN
-F 1 "GND" V 2355 1672 50  0000 R CNN
-F 2 "" H 2350 1800 50  0001 C CNN
-F 3 "" H 2350 1800 50  0001 C CNN
-	1    2350 1800
+P 2450 1700
+F 0 "#PWR0105" H 2450 1450 50  0001 C CNN
+F 1 "GND" V 2455 1572 50  0000 R CNN
+F 2 "" H 2450 1700 50  0001 C CNN
+F 3 "" H 2450 1700 50  0001 C CNN
+	1    2450 1700
 	0    1    1    0
 $EndComp
@@
 L power:GND #PWR0106
 U 1 1 5AD32478
-P 3850 1800
-F 0 "#PWR0106" H 3850 1550 50  0001 C CNN
-F 1 "GND" V 3855 1672 50  0000 R CNN
-F 2 "" H 3850 1800 50  0001 C CNN
-F 3 "" H 3850 1800 50  0001 C CNN
-	1    3850 1800
+P 3950 1700
+F 0 "#PWR0106" H 3950 1450 50  0001 C CNN
+F 1 "GND" V 3955 1572 50  0000 R CNN
+F 2 "" H 3950 1700 50  0001 C CNN
+F 3 "" H 3950 1700 50  0001 C CNN
+	1    3950 1700
 	0    1    1    0
 $EndComp
@@
 Wire Wire Line
 	1150 4450 1150 4700
-NoConn ~ 4850 1500
-NoConn ~ 4850 1600
-NoConn ~ 4850 1700
-NoConn ~ 4850 1800
-NoConn ~ 4850 1900
+NoConn ~ 4750 1400
+NoConn ~ 4750 1500
+NoConn ~ 4750 1600
+NoConn ~ 4750 1700
+NoConn ~ 4750 1800
 $Comp
 L power:GND #PWR0111
@@
 L power:GND #PWR0114
 U 1 1 5AD33A61
-P 4350 2400
-F 0 "#PWR0114" H 4350 2150 50  0001 C CNN
-F 1 "GND" H 4355 2227 50  0000 C CNN
-F 2 "" H 4350 2400 50  0001 C CNN
-F 3 "" H 4350 2400 50  0001 C CNN
-	1    4350 2400
+P 4350 2200
+F 0 "#PWR0114" H 4350 1950 50  0001 C CNN
+F 1 "GND" H 4355 2027 50  0000 C CNN
+F 2 "" H 4350 2200 50  0001 C CNN
+F 3 "" H 4350 2200 50  0001 C CNN
+	1    4350 2200
 	1    0    0    -1
 $EndComp
@@
 L power:GND #PWR0115
 U 1 1 5AD33A82
-P 2850 2400
-F 0 "#PWR0115" H 2850 2150 50  0001 C CNN
-F 1 "GND" H 2855 2227 50  0000 C CNN
-F 2 "" H 2850 2400 50  0001 C CNN
-F 3 "" H 2850 2400 50  0001 C CNN
-	1    2850 2400
+P 2850 2200
+F 0 "#PWR0115" H 2850 1950 50  0001 C CNN
+F 1 "GND" H 2855 2027 50  0000 C CNN
+F 2 "" H 2850 2200 50  0001 C CNN
+F 3 "" H 2850 2200 50  0001 C CNN
+	1    2850 2200
 	1    0    0    -1
 $EndComp
@@
 L power:GND #PWR0116
 U 1 1 5AD33ADA
-P 1300 2400
-F 0 "#PWR0116" H 1300 2150 50  0001 C CNN
-F 1 "GND" H 1305 2227 50  0000 C CNN
-F 2 "" H 1300 2400 50  0001 C CNN
-F 3 "" H 1300 2400 50  0001 C CNN
-	1    1300 2400
+P 1300 2200
+F 0 "#PWR0116" H 1300 1950 50  0001 C CNN
+F 1 "GND" H 1305 2027 50  0000 C CNN
+F 2 "" H 1300 2200 50  0001 C CNN
+F 3 "" H 1300 2200 50  0001 C CNN
+	1    1300 2200
 	1    0    0    -1
 $EndComp
@@
 Wire Wire Line
 	1450 5800 1450 6050
+$Comp
+L 74xx:74HC595 U1
+U 1 1 5B34E9D4
+P 1300 1500
+F 0 "U1" H 1300 1500 50  0000 C CNN
+F 1 "74HC595" H 1300 1150 50  0000 C CNN
+F 2 "" H 1300 1500 50  0001 C CNN
+F 3 "http://www.ti.com/lit/ds/symlink/sn74hc595.pdf" H 1300 1500 50  0001 C CNN
+	1    1300 1500
+	1    0    0    -1
+$EndComp
+Wire Wire Line
+	1700 2000 1950 2000
+$Comp
+L 74xx:74HC595 U2
+U 1 1 5B34F6A3
+P 2850 1500
+F 0 "U2" H 2850 1500 50  0000 C CNN
+F 1 "74HC595" H 2850 1150 50  0000 C CNN
+F 2 "" H 2850 1500 50  0001 C CNN
+F 3 "http://www.ti.com/lit/ds/symlink/sn74hc595.pdf" H 2850 1500 50  0001 C CNN
+	1    2850 1500
+	1    0    0    -1
+$EndComp
+$Comp
+L 74xx:74HC595 U3
+U 1 1 5B34F82B
+P 4350 1500
+F 0 "U3" H 4350 1450 50  0000 C CNN
+F 1 "74HC595" H 4350 1200 50  0000 C CNN
+F 2 "" H 4350 1500 50  0001 C CNN
+F 3 "http://www.ti.com/lit/ds/symlink/sn74hc595.pdf" H 4350 1500 50  0001 C CNN
+	1    4350 1500
+	1    0    0    -1
+$EndComp
+Wire Wire Line
+	1950 1100 2450 1100
+Wire Wire Line
+	3500 1100 3950 1100
 $EndSCHEMATC

Commit message: Updates.
Changed lines of the file:
@@
 L power:+5V #PWR0103
 U 1 1 5AD3213B
-P 800 1500
-F 0 "#PWR0103" H 800 1350 50  0001 C CNN
-F 1 "+5V" V 815 1628 50  0000 L CNN
-F 2 "" H 800 1500 50  0001 C CNN
-F 3 "" H 800 1500 50  0001 C CNN
-	1    800  1500
+P 900 1400
+F 0 "#PWR0103" H 900 1250 50  0001 C CNN
+F 1 "+5V" V 915 1528 50  0000 L CNN
+F 2 "" H 900 1400 50  0001 C CNN
+F 3 "" H 900 1400 50  0001 C CNN
+	1    900  1400
 	0    -1   -1   0
 $EndComp
-Text Label 800  1200 2    50   ~ 0
+Text Label 900  1100 2    50   ~ 0
 SER
 Text Label 1450 3850 2    50   ~ 0
@@
 Text Label 1450 3950 2    50   ~ 0
 SRCLK
-Text Label 800  1400 2    50   ~ 0
+Text Label 900  1300 2    50   ~ 0
 SRCLK
 Text Label 2450 1300 2    50   ~ 0
@@
 Text Label 1450 4050 2    50   ~ 0
 RCLK
-Text Label 800  1700 2    50   ~ 0
+Text Label 900  1600 2    50   ~ 0
 RCLK
 Text Label 2450 1600 2    50   ~ 0
@@
 L power:GND #PWR0104
 U 1 1 5AD32424
-P 800 1800
-F 0 "#PWR0104" H 800 1550 50  0001 C CNN
-F 1 "GND" V 805 1672 50  0000 R CNN
-F 2 "" H 800 1800 50  0001 C CNN
-F 3 "" H 800 1800 50  0001 C CNN
-	1    800  1800
+P 900 1700
+F 0 "#PWR0104" H 900 1450 50  0001 C CNN
+F 1 "GND" V 905 1572 50  0000 R CNN
+F 2 "" H 900 1700 50  0001 C CNN
+F 3 "" H 900 1700 50  0001 C CNN
+	1    900  1700
 	0    1    1    0
 $EndComp
